Commit message: fixed typo in inertia properties of the hippo2 model

File: urdf/hippo2_params.xacro (robot description, xacro)
@@ -3,5 +3,5 @@
     <xacro:property name="base_mass" value="1.47" />
     <xacro:property name="ixx" value="0.0024" />
-    <xacro:property name="iyy" value="0.01717" />
+    <xacro:property name="iyy" value="0.010717" />
     <xacro:property name="izz" value="0.010717" />
 </robot>
