Commit message: added xacro params for thrusters

File: urdf/thruster_macro.xacro (robot description, xacro)
@@ -2,4 +2,5 @@
 <robot xmlns:xacro="http://www.ros.org/wiki/xacro">
     <xacro:macro name="thruster" params="suffix parent xyz axis cw">
+        <xacro:include filename="$(find hippo_sim)/urdf/thruster_params.xacro" />
         <xacro:property name="mount_link" value="${suffix}_thruster_mount_link" />
         <xacro:property name="mount_joint" value="${suffix}_thruster_mount_joint" />
@@ -11,6 +12,6 @@
             <origin xyz="0 0 0" rpy="0 0 0" />
             <inertial>
-                <mass value="${base_mass}" />
-                <inertia ixx="${ixx}" ixy="0.0" ixz="0.0" iyy="${iyy}" iyz="0.0" izz="${izz}" />
+                <mass value="${thruster_mass}" />
+                <inertia ixx="${thruster_ixx}" ixy="0.0" ixz="0.0" iyy="${thruster_iyy}" iyz="0.0" izz="${thruster_izz}" />
             </inertial>
             <visual>
@@ -46,6 +47,6 @@
             <origin xyz="0 0 0" rpy="0 0 0" />
             <inertial>
-                <mass value="${base_mass}" />
-                <inertia ixx="${ixx}" ixy="0.0" ixz="0.0" iyy="${iyy}" iyz="0.0" izz="${izz}" />
+                <mass value="${thruster_mass}" />
+                <inertia ixx="${thruster_ixx}" ixy="0.0" ixz="0.0" iyy="${thruster_iyy}" iyz="0.0" izz="${thruster_izz}" />
             </inertial>
             <visual>
@@ -81,6 +82,6 @@
             <origin xyz="0 0 0" rpy="0 0 0" />
             <inertial>
-                <mass value="${base_mass}" />
-                <inertia ixx="${ixx}" ixy="0.0" ixz="0.0" iyy="${iyy}" iyz="0.0" izz="${izz}" />
+                <mass value="${thruster_mass}" />
+                <inertia ixx="${thruster_ixx}" ixy="0.0" ixz="0.0" iyy="${thruster_iyy}" iyz="0.0" izz="${thruster_izz}" />
             </inertial>
             <visual>

Commit message: added thruster plugin

File: urdf/thruster_macro.xacro (robot description, xacro)
@@ -91,4 +91,17 @@
             </visual>
         </link>
+        <gazebo>
+            <plugin filename="ThrusterPlugin" name="ignition::gazebo::systems::ThrusterPlugin">
+                <thruster_config>
+                    <link>${propeller_link}</link>
+                    <joint>${propeller_joint}</joint>
+                    <linear_coeff>1e-5</linear_coeff>
+                    <quadratic_coeff>1e-5</quadratic_coeff>
+                    <torque_coeff>0.0024</torque_coeff>
+                    <rpm_scaler>10.0</rpm_scaler>
+                    <max_rpm>800</max_rpm>
+                </thruster_config>
+            </plugin>
+        </gazebo>
         <gazebo reference="${propeller_link}">
             <visual>

Commit message: thruster mount joint is now static

File: urdf/thruster_macro.xacro (robot description, xacro)
@@ -38,5 +38,5 @@
             </visual>
         </gazebo>
-        <joint name="${mount_joint}" type="continuous">
+        <joint name="${mount_joint}" type="fixed">
             <axis xyz="${axis}" />
             <origin xyz="${xyz}" />
@@ -44,4 +44,8 @@
             <child link="${mount_link}" />
         </joint>
+        <gazebo reference="${mount_joint}">
+            <disableFixedJointLumping>true</disableFixedJointLumping>
+            <preserveFixedJoint>true</preserveFixedJoint>
+        </gazebo>
         <link name="${hull_link}">
             <origin xyz="0 0 0" rpy="0 0 0" />

Commit message: introduced thruster plugin properties

File: urdf/thruster_macro.xacro (robot description, xacro)
@@ -100,9 +100,9 @@
                     <link>${propeller_link}</link>
                     <joint>${propeller_joint}</joint>
-                    <linear_coeff>1e-5</linear_coeff>
-                    <quadratic_coeff>1e-5</quadratic_coeff>
-                    <torque_coeff>0.0024</torque_coeff>
-                    <rpm_scaler>10.0</rpm_scaler>
-                    <max_rpm>800</max_rpm>
+                    <linear_coeff>${thrust_linear_coeff}</linear_coeff>
+                    <quadratic_coeff>${thrust_quadratic_coeff}</quadratic_coeff>
+                    <torque_coeff>${torque_constant}</torque_coeff>
+                    <rpm_scaler>${rpm_scaler}</rpm_scaler>
+                    <max_rpm>${max_rpm}</max_rpm>
                 </thruster_config>
             </plugin>

File: urdf/thruster_params.xacro (robot description, xacro)
@@ -5,3 +5,8 @@
     <xacro:property name="thruster_iyy" value="1e-6" />
     <xacro:property name="thruster_izz" value="1e-6" />
+    <xacro:property name="thrust_linear_coeff" value="15.89" />
+    <xacro:property name="thrust_quadratic_coeff" value="23.2" />
+    <xacro:property name="torque_constant" value="10.0" />
+    <xacro:property name="rpm_scaler" value="10.0" />
+    <xacro:property name="max_rpm" value="800" />
 </robot>

Commit message: added first-order model for thrusters

File: urdf/thruster_macro.xacro (robot description, xacro)
@@ -48,5 +48,5 @@
             <preserveFixedJoint>true</preserveFixedJoint>
         </gazebo>
-        <!-- <link name="${hull_link}">
+        <link name="${hull_link}">
             <origin xyz="0 0 0" rpy="0 0 0" />
             <inertial>
@@ -82,5 +82,5 @@
             <parent link="${parent}" />
             <child link="${hull_link}" />
-        </joint> -->
+        </joint>
         <link name="${propeller_link}">
             <origin xyz="0 0 0" rpy="0 0 0" />
@@ -108,4 +108,6 @@
                     <turning_direction>${turning_direction}</turning_direction>
                     <propeller_direction>${propeller_direction}</propeller_direction>
+                    <timeconstant_up>${timeconstant_up}</timeconstant_up>
+                    <timeconstant_down>${timeconstant_down}</timeconstant_down>
                 </thruster_config>
             </plugin>

File: urdf/thruster_params.xacro (robot description, xacro)
@@ -5,8 +5,10 @@
     <xacro:property name="thruster_iyy" value="1e-6" />
     <xacro:property name="thruster_izz" value="1e-6" />
-    <xacro:property name="thrust_linear_coeff" value="15.89e-2" />
-    <xacro:property name="thrust_quadratic_coeff" value="23.2e-2" />
+    <xacro:property name="thrust_linear_coeff" value="15.89e-5" />
+    <xacro:property name="thrust_quadratic_coeff" value="23.2e-5" />
     <xacro:property name="torque_constant" value="1e-2" />
     <xacro:property name="rpm_scaler" value="1" />
     <xacro:property name="max_rpm" value="800" />
+    <xacro:property name="timeconstant_up" value="1.0" />
+    <xacro:property name="timeconstant_down" value="1.0" />
 </robot>
