Commit message: fixed wrong visual tag

File: urdf/hippo2.xacro (robot description, xacro)
@@ -13,5 +13,7 @@
         </inertial>
         <visual>
-            <mesh filename="package://hippo_sim/meshes/hippo2.stl" />
+            <geometry>
+                <mesh filename="file://$(find hippo_sim)/meshes/hippo2.dae" />
+            </geometry>
         </visual>
     </link>

Commit message: added meshfiles

File: urdf/hippo2.xacro (robot description, xacro)
@@ -14,8 +14,103 @@
         <visual>
             <geometry>
-                <mesh filename="file://$(find hippo_sim)/meshes/hippo2.dae" />
+                <mesh filename="$(find hippo_sim)/meshes/hippo3_motor_hull.dae" />
             </geometry>
         </visual>
     </link>
+    <link name="base_link2">
+        <origin> xyz="0 0 0" rpy="0 0 0"</origin>
+        <inertial>
+            <mass value="${base_mass}" />
+            <inertia ixx="${ixx}" ixy="0.0" ixz="0.0" iyy="${iyy}" iyz="0.0" izz="${izz}" />
+        </inertial>
+        <visual>
+            <geometry>
+                <mesh filename="$(find hippo_sim)/meshes/hippo3_motor_mount.dae" />
+            </geometry>
+        </visual>
+    </link>
+    <joint name="joint" type="fixed">
+        <parent link="base_link"/>
+        <child link="base_link2" />
+    </joint>
+    <link name="base_link3">
+        <origin> xyz="0 0 0" rpy="0 0 0"</origin>
+        <inertial>
+            <mass value="${base_mass}" />
+            <inertia ixx="${ixx}" ixy="0.0" ixz="0.0" iyy="${iyy}" iyz="0.0" izz="${izz}" />
+        </inertial>
+        <visual>
+            <geometry>
+                <mesh filename="$(find hippo_sim)/meshes/propeller.dae" />
+            </geometry>
+        </visual>
+    </link>
+    <joint name="joint2" type="fixed">
+        <parent link="base_link"/>
+        <child link="base_link3" />
+    </joint>
     <xacro:thruster parent="base_link" suffix="starboard_top" xyz="0 0.1 0.1" axis="1 0 0" cw="true" />
+    <gazebo reference="joint">
+        <preserveFixedJoint>true</preserveFixedJoint>
+    </gazebo>
+    <gazebo reference="joint2">
+        <preserveFixedJoint>true</preserveFixedJoint>
+    </gazebo>
+    <gazebo reference="base_link">
+        <visual>
+            <material>
+                <ambient>1 1 1 1</ambient>
+                <diffuse>1 1 1 1</diffuse>
+                <specular>1 1 1 1</specular>
+                <pbr>
+                    <metal>
+                        <metalness>1</metalness>
+                        <roughness>0.5</roughness>
+                        <environment_map>$(find hippo_sim)/textures/env_map.dds</environment_map>
+                        <!-- <ambient_occlusion_map>$(find hippo_sim)/textures/albedo.png</ambient_occlusion_map> -->
+                        <!-- <normal_map tpye="tangent">$(find hippo_sim)/textures/normal.png</normal_map> -->
+                        <albedo_map>$(find hippo_sim)/textures/hippocampus_text.png</albedo_map>
+                    </metal>
+                </pbr>
+            </material>
+        </visual>
+    </gazebo>
+    <gazebo reference="base_link2">
+        <visual>
+            <material>
+                <ambient>1 1 1 1</ambient>
+                <diffuse>1 1 1 1</diffuse>
+                <specular>1 1 1 1</specular>
+                <pbr>
+                    <metal>
+                        <metalness>1</metalness>
+                        <roughness>0.5</roughness>
+                        <environment_map>$(find hippo_sim)/textures/env_map.dds</environment_map>
+                        <!-- <ambient_occlusion_map>$(find hippo_sim)/textures/albedo.png</ambient_occlusion_map> -->
+                        <!-- <normal_map tpye="tangent">$(find hippo_sim)/textures/normal.png</normal_map> -->
+                        <albedo_map>$(find hippo_sim)/textures/grey.png</albedo_map>
+                    </metal>
+                </pbr>
+            </material>
+        </visual>
+    </gazebo>
+    <gazebo reference="base_link3">
+        <visual>
+            <material>
+                <ambient>1 1 1 1</ambient>
+                <diffuse>1 1 1 1</diffuse>
+                <specular>1 1 1 1</specular>
+                <pbr>
+                    <metal>
+                        <metalness>1</metalness>
+                        <roughness>0.3</roughness>
+                        <environment_map>$(find hippo_sim)/textures/env_map.dds</environment_map>
+                        <!-- <ambient_occlusion_map>$(find hippo_sim)/textures/albedo.png</ambient_occlusion_map> -->
+                        <!-- <normal_map tpye="tangent">$(find hippo_sim)/textures/normal.png</normal_map> -->
+                        <albedo_map>$(find hippo_sim)/textures/red.png</albedo_map>
+                    </metal>
+                </pbr>
+            </material>
+        </visual>
+    </gazebo>
 </robot>

Commit message: added meshfiles and updated thruster macro

File: urdf/hippo2.xacro (robot description, xacro)
@@ -14,45 +14,42 @@
         <visual>
             <geometry>
-                <mesh filename="$(find hippo_sim)/meshes/hippo3_motor_hull.dae" />
+                <mesh filename="$(find hippo_sim)/meshes/hippo3_tube.dae" />
             </geometry>
         </visual>
     </link>
-    <link name="base_link2">
-        <origin> xyz="0 0 0" rpy="0 0 0"</origin>
+    <link name="flange_link">
         <inertial>
-            <mass value="${base_mass}" />
-            <inertia ixx="${ixx}" ixy="0.0" ixz="0.0" iyy="${iyy}" iyz="0.0" izz="${izz}" />
+            <mass value="1e-5" />
+            <inertia ixx="1e-5" ixy="0.0" ixz="0.0" iyy="1e-5" iyz="0.0" izz="1e-5" />
         </inertial>
         <visual>
             <geometry>
-                <mesh filename="$(find hippo_sim)/meshes/hippo3_motor_mount.dae" />
+                <mesh filename="$(find hippo_sim)/meshes/hippo3_flange.dae" />
             </geometry>
         </visual>
     </link>
-    <joint name="joint" type="fixed">
-        <parent link="base_link"/>
-        <child link="base_link2" />
+    <joint name="flange_joint" type="fixed">
+        <parent link="base_link" />
+        <child link="flange_link" />
     </joint>
-    <link name="base_link3">
-        <origin> xyz="0 0 0" rpy="0 0 0"</origin>
+    <link name="dome_link">
         <inertial>
-            <mass value="${base_mass}" />
-            <inertia ixx="${ixx}" ixy="0.0" ixz="0.0" iyy="${iyy}" iyz="0.0" izz="${izz}" />
+            <mass value="1e-5" />
+            <inertia ixx="1e-5" ixy="0.0" ixz="0.0" iyy="1e-5" iyz="0.0" izz="1e-5" />
         </inertial>
         <visual>
             <geometry>
-                <mesh filename="$(find hippo_sim)/meshes/propeller.dae" />
+                <mesh filename="$(find hippo_sim)/meshes/hippo3_dome.dae" />
             </geometry>
         </visual>
     </link>
-    <joint name="joint2" type="fixed">
-        <parent link="base_link"/>
-        <child link="base_link3" />
+    <joint name="dome_joint" type="fixed">
+        <parent link="base_link" />
+        <child link="dome_link" />
     </joint>
-    <xacro:thruster parent="base_link" suffix="starboard_top" xyz="0 0.1 0.1" axis="1 0 0" cw="true" />
-    <gazebo reference="joint">
+    <gazebo reference="flange_joint">
         <preserveFixedJoint>true</preserveFixedJoint>
     </gazebo>
-    <gazebo reference="joint2">
+    <gazebo reference="dome_joint">
         <preserveFixedJoint>true</preserveFixedJoint>
     </gazebo>
@@ -60,15 +57,22 @@
         <visual>
             <material>
+                <ambient>0.5 0.5 0.9 0.2</ambient>
+                <diffuse>0.5 0.5 0.9 0.5</diffuse>
+                <specular>1 1 1 1</specular>
+            </material>
+        </visual>
+    </gazebo>
+    <gazebo reference="flange_link">
+        <visual>
+            <material>
                 <ambient>1 1 1 1</ambient>
                 <diffuse>1 1 1 1</diffuse>
                 <specular>1 1 1 1</specular>
-                <pbr>
+                <pbr>grey
                     <metal>
                         <metalness>1</metalness>
                         <roughness>0.5</roughness>
                         <environment_map>$(find hippo_sim)/textures/env_map.dds</environment_map>
-                        <!-- <ambient_occlusion_map>$(find hippo_sim)/textures/albedo.png</ambient_occlusion_map> -->
-                        <!-- <normal_map tpye="tangent">$(find hippo_sim)/textures/normal.png</normal_map> -->
-                        <albedo_map>$(find hippo_sim)/textures/hippocampus_text.png</albedo_map>
+                        <albedo_map>$(find hippo_sim)/textures/dark_grey.png</albedo_map>
                     </metal>
                 </pbr>
@@ -76,41 +80,16 @@
         </visual>
     </gazebo>
-    <gazebo reference="base_link2">
+    <gazebo reference="dome_link">
         <visual>
             <material>
-                <ambient>1 1 1 1</ambient>
-                <diffuse>1 1 1 1</diffuse>
+                <ambient>0.5 0.5 0.9 0.2</ambient>
+                <diffuse>0.5 0.5 0.9 0.5</diffuse>
                 <specular>1 1 1 1</specular>
-                <pbr>
-                    <metal>
-                        <metalness>1</metalness>
-                        <roughness>0.5</roughness>
-                        <environment_map>$(find hippo_sim)/textures/env_map.dds</environment_map>
-                        <!-- <ambient_occlusion_map>$(find hippo_sim)/textures/albedo.png</ambient_occlusion_map> -->
-                        <!-- <normal_map tpye="tangent">$(find hippo_sim)/textures/normal.png</normal_map> -->
-                        <albedo_map>$(find hippo_sim)/textures/grey.png</albedo_map>
-                    </metal>
-                </pbr>
             </material>
         </visual>
     </gazebo>
-    <gazebo reference="base_link3">
-        <visual>
-            <material>
-                <ambient>1 1 1 1</ambient>
-                <diffuse>1 1 1 1</diffuse>
-                <specular>1 1 1 1</specular>
-                <pbr>
-                    <metal>
-                        <metalness>1</metalness>
-                        <roughness>0.3</roughness>
-                        <environment_map>$(find hippo_sim)/textures/env_map.dds</environment_map>
-                        <!-- <ambient_occlusion_map>$(find hippo_sim)/textures/albedo.png</ambient_occlusion_map> -->
-                        <!-- <normal_map tpye="tangent">$(find hippo_sim)/textures/normal.png</normal_map> -->
-                        <albedo_map>$(find hippo_sim)/textures/red.png</albedo_map>
-                    </metal>
-                </pbr>
-            </material>
-        </visual>
-    </gazebo>
+    <xacro:thruster parent="base_link" suffix="port_top" xyz="0 -${thruster_r / 2**0.5} ${thruster_r / 2**0.5}" axis="1 0 0" cw="true" />
+    <xacro:thruster parent="base_link" suffix="starboard_top" xyz="0 ${thruster_r / 2**0.5} ${thruster_r / 2**0.5}" axis="1 0 0" cw="false" />
+    <xacro:thruster parent="base_link" suffix="starboard_bot" xyz="0 ${thruster_r / 2**0.5} -${thruster_r / 2**0.5}" axis="1 0 0" cw="true" />
+    <xacro:thruster parent="base_link" suffix="port_bot" xyz="0 -${thruster_r / 2**0.5} -${thruster_r / 2**0.5}" axis="1 0 0" cw="false" />
 </robot>

File: urdf/hippo2_params.xacro (robot description, xacro)
@@ -5,3 +5,4 @@
     <xacro:property name="iyy" value="0.010717" />
     <xacro:property name="izz" value="0.010717" />
+    <xacro:property name="thruster_r" value="0.09" />
 </robot>

File: urdf/thruster_macro.xacro (robot description, xacro)
@@ -2,18 +2,115 @@
 <robot xmlns:xacro="http://www.ros.org/wiki/xacro">
     <xacro:macro name="thruster" params="suffix parent xyz axis cw">
-        <joint name="${suffix}_thruster_joint" type="continuous">
+        <xacro:property name="mount_link" value="${suffix}_thruster_mount_link" />
+        <xacro:property name="mount_joint" value="${suffix}_thruster_mount_joint" />
+        <xacro:property name="hull_link" value="${suffix}_thruster_hull_link" />
+        <xacro:property name="hull_joint" value="${suffix}_thruster_hull_joint" />
+        <xacro:property name="propeller_link" value="${suffix}_thruster_propeller_link" />
+        <xacro:property name="propeller_joint" value="${suffix}_thruster_propeller_joint" />
+        <link name="${mount_link}">
+            <origin xyz="0 0 0" rpy="0 0 0" />
+            <inertial>
+                <mass value="${base_mass}" />
+                <inertia ixx="${ixx}" ixy="0.0" ixz="0.0" iyy="${iyy}" iyz="0.0" izz="${izz}" />
+            </inertial>
+            <visual>
+                <geometry>
+                    <mesh filename="$(find hippo_sim)/meshes/hippo3_motor_mount.dae" />
+                </geometry>
+            </visual>
+        </link>
+        <gazebo reference="${mount_link}">
+            <visual>
+                <material>
+                    <ambient>1 1 1 1</ambient>
+                    <diffuse>1 1 1 1</diffuse>
+                    <specular>1 1 1 1</specular>
+                    <pbr>
+                        <metal>
+                            <metalness>1</metalness>
+                            <roughness>0.5</roughness>
+                            <environment_map>$(find hippo_sim)/textures/env_map.dds</environment_map>
+                            <albedo_map>$(find hippo_sim)/textures/grey.png</albedo_map>
+                        </metal>
+                    </pbr>
+                </material>
+            </visual>
+        </gazebo>
+        <joint name="${mount_joint}" type="continuous">
             <axis xyz="${axis}" />
             <origin xyz="${xyz}" />
             <parent link="${parent}" />
-            <child link="${suffix}_thruster_link" />
+            <child link="${mount_link}" />
         </joint>
-        <link name="${suffix}_thruster_link">
+        <link name="${hull_link}">
             <origin xyz="0 0 0" rpy="0 0 0" />
+            <inertial>
+                <mass value="${base_mass}" />
+                <inertia ixx="${ixx}" ixy="0.0" ixz="0.0" iyy="${iyy}" iyz="0.0" izz="${izz}" />
+            </inertial>
             <visual>
                 <geometry>
-                    <mesh filename="package://hippo_sim/meshes/propeller.stl" />
+                    <mesh filename="$(find hippo_sim)/meshes/hippo3_motor_hull.dae" />
                 </geometry>
             </visual>
         </link>
+        <gazebo reference="${hull_link}">
+            <visual>
+                <material>
+                    <ambient>1 1 1 1</ambient>
+                    <diffuse>1 1 1 1</diffuse>
+                    <specular>1 1 1 1</specular>
+                    <pbr>
+                        <metal>
+                            <metalness>1</metalness>
+                            <roughness>0.5</roughness>
+                            <environment_map>$(find hippo_sim)/textures/env_map.dds</environment_map>
+                            <albedo_map>$(find hippo_sim)/textures/hippocampus_text.png</albedo_map>
+                        </metal>
+                    </pbr>
+                </material>
+            </visual>
+        </gazebo>
+        <joint name="${hull_joint}" type="continuous">
+            <axis xyz="${axis}" />
+            <origin xyz="${xyz}" />
+            <parent link="${parent}" />
+            <child link="${hull_link}" />
+        </joint>
+        <link name="${propeller_link}">
+            <origin xyz="0 0 0" rpy="0 0 0" />
+            <inertial>
+                <mass value="${base_mass}" />
+                <inertia ixx="${ixx}" ixy="0.0" ixz="0.0" iyy="${iyy}" iyz="0.0" izz="${izz}" />
+            </inertial>
+            <visual>
+                <geometry>
+                    <mesh filename="$(find hippo_sim)/meshes/propeller.dae" />
+                </geometry>
+            </visual>
+        </link>
+        <gazebo reference="${propeller_link}">
+            <visual>
+                <material>
+                    <ambient>1 1 1 1</ambient>
+                    <diffuse>1 1 1 1</diffuse>
+                    <specular>1 1 1 1</specular>
+                    <pbr>
+                        <metal>
+                            <metalness>1</metalness>
+                            <roughness>0.3</roughness>
+                            <environment_map>$(find hippo_sim)/textures/env_map.dds</environment_map>
+                            <albedo_map>$(find hippo_sim)/textures/red.png</albedo_map>
+                        </metal>
+                    </pbr>
+                </material>
+            </visual>
+        </gazebo>
+        <joint name="${propeller_joint}" type="continuous">
+            <axis xyz="${axis}" />
+            <origin xyz="${xyz}" />
+            <parent link="${parent}" />
+            <child link="${propeller_link}" />
+        </joint>
     </xacro:macro>
 </robot>

Commit message: added imu

File: urdf/hippo2.xacro (robot description, xacro)
@@ -4,8 +4,7 @@
     <xacro:include filename="$(find hippo_sim)/urdf/thruster_macro.xacro" />
     <gazebo>
-        <static>true</static>
+        <static>false</static>
     </gazebo>
     <link name="base_link">
-        <origin> xyz="0 0 0" rpy="0 0 0"</origin>
         <inertial>
             <mass value="${base_mass}" />
@@ -55,4 +54,9 @@
     </gazebo>
     <gazebo reference="base_link">
+        <sensor name="imu_sensor" type="imu">
+            <always_on>1</always_on>
+            <visualize>true</visualize>
+            <topic>imu_topic</topic>
+        </sensor>
         <visual>
             <material>

Commit message: added buoyancy plugin

File: urdf/hippo2.xacro (robot description, xacro)
@@ -98,3 +98,15 @@
     <xacro:thruster parent="base_link" suffix="starboard_bot" xyz="0 ${thruster_r / 2**0.5} -${thruster_r / 2**0.5}" axis="1 0 0" cw="true" />
     <xacro:thruster parent="base_link" suffix="port_bot" xyz="0 -${thruster_r / 2**0.5} -${thruster_r / 2**0.5}" axis="1 0 0" cw="false" />
+    <gazebo>
+        <plugin filename="BuoyancyPlugin"
+        name="ignition::gazebo::systems::BuoyancyPlugin">
+        <buoyancy>
+            <link_name>base_link</link_name>
+            <origin>0 0 0.002</origin>
+            <force_added>0</force_added>
+            <compensation>1.01</compensation>
+            <height_scale_limit>0.1</height_scale_limit>
+        </buoyancy>
+      </plugin>
+    </gazebo>
 </robot>

Commit message: added hydrodynamics plugin

File: urdf/hippo2.xacro (robot description, xacro)
@@ -109,4 +109,14 @@
         </buoyancy>
       </plugin>
+      <plugin filename="HydrodynamicsPlugin"
+      name="ignition::gazebo::systems::HydrodynamicsPlugin">
+      <hydrodynamics>
+        <link>base_link</link>
+        <added_mass_linear>1.11 2.8 2.8</added_mass_linear>
+        <added_mass_angular>0.00451 0.0163 0.0163</added_mass_angular>
+        <damping_linear>5.39 17.36 17.36</damping_linear>
+        <damping_angular>0.00114 0.007 0.007</damping_angular>
+      </hydrodynamics>
+    </plugin>
     </gazebo>
 </robot>

Commit message: replaced hydrodynamic parameters with properties

File: urdf/hippo2.xacro (robot description, xacro)
@@ -74,5 +74,4 @@
                 <specular>1 1 1 1</specular>
                 <pbr>
-                    grey
                     <metal>
                         <metalness>1</metalness>
@@ -113,8 +112,8 @@
       <hydrodynamics>
         <link>base_link</link>
-        <added_mass_linear>1.11 2.8 2.8</added_mass_linear>
-        <added_mass_angular>0.00451 0.0163 0.0163</added_mass_angular>
-        <damping_linear>5.39 17.36 17.36</damping_linear>
-        <damping_angular>0.00114 0.007 0.007</damping_angular>
+        <added_mass_linear>${added_mass_linear}</added_mass_linear>
+        <added_mass_angular>${added_mass_angular}</added_mass_angular>
+        <damping_linear>${damping_linear}</damping_linear>
+        <damping_angular>${damping_angular}</damping_angular>
       </hydrodynamics>
     </plugin>

File: urdf/hippo2_params.xacro (robot description, xacro)
@@ -6,3 +6,7 @@
     <xacro:property name="izz" value="0.010717" />
     <xacro:property name="thruster_r" value="0.09" />
+    <xacro:property name="added_mass_linear" value="1.11 2.8 2.8" />
+    <xacro:property name="added_mass_angular" value="0.00451 0.0163 0.0163"/>
+    <xacro:property name="damping_linear" value="5.39 17.36 17.36"/>
+    <xacro:property name="damping_angular" value="0.00174 0.007 0.007"/>
 </robot>
