Commit message: thruster plugin applies force

File: urdf/hippo2.xacro (robot description, xacro)
@@ -93,29 +93,27 @@
         </visual>
     </gazebo>
-    <xacro:thruster parent="base_link" suffix="port_top" xyz="0 -${thruster_r / 2**0.5} ${thruster_r / 2**0.5}" axis="1 0 0" cw="true" />
-    <xacro:thruster parent="base_link" suffix="starboard_top" xyz="0 ${thruster_r / 2**0.5} ${thruster_r / 2**0.5}" axis="1 0 0" cw="false" />
-    <xacro:thruster parent="base_link" suffix="starboard_bot" xyz="0 ${thruster_r / 2**0.5} -${thruster_r / 2**0.5}" axis="1 0 0" cw="true" />
-    <xacro:thruster parent="base_link" suffix="port_bot" xyz="0 -${thruster_r / 2**0.5} -${thruster_r / 2**0.5}" axis="1 0 0" cw="false" />
+    <xacro:thruster parent="base_link" suffix="port_top" xyz="0 -${thruster_r / 2**0.5} ${thruster_r / 2**0.5}" axis="1 0 0" cw="true" color="red" number="0" />
+    <xacro:thruster parent="base_link" suffix="starboard_top" xyz="0 ${thruster_r / 2**0.5} ${thruster_r / 2**0.5}" axis="1 0 0" cw="false" color="green" number="1" />
+    <xacro:thruster parent="base_link" suffix="starboard_bot" xyz="0 ${thruster_r / 2**0.5} -${thruster_r / 2**0.5}" axis="1 0 0" cw="true" color="grey" number="2" />
+    <xacro:thruster parent="base_link" suffix="port_bot" xyz="0 -${thruster_r / 2**0.5} -${thruster_r / 2**0.5}" axis="1 0 0" cw="false" color="grey" number="3" />
     <gazebo>
-        <plugin filename="BuoyancyPlugin"
-        name="ignition::gazebo::systems::BuoyancyPlugin">
-        <buoyancy>
-            <link_name>base_link</link_name>
-            <origin>0 0 0.002</origin>
-            <force_added>0</force_added>
-            <compensation>1.01</compensation>
-            <height_scale_limit>0.1</height_scale_limit>
-        </buoyancy>
-      </plugin>
-      <plugin filename="HydrodynamicsPlugin"
-      name="ignition::gazebo::systems::HydrodynamicsPlugin">
-      <hydrodynamics>
-        <link>base_link</link>
-        <added_mass_linear>${added_mass_linear}</added_mass_linear>
-        <added_mass_angular>${added_mass_angular}</added_mass_angular>
-        <damping_linear>${damping_linear}</damping_linear>
-        <damping_angular>${damping_angular}</damping_angular>
-      </hydrodynamics>
-    </plugin>
+        <plugin filename="BuoyancyPlugin" name="ignition::gazebo::systems::BuoyancyPlugin">
+            <buoyancy>
+                <link_name>base_link</link_name>
+                <origin>0 0 0.002</origin>
+                <force_added>0</force_added>
+                <compensation>1.01</compensation>
+                <height_scale_limit>0.1</height_scale_limit>
+            </buoyancy>
+        </plugin>
+        <plugin filename="HydrodynamicsPlugin" name="ignition::gazebo::systems::HydrodynamicsPlugin">
+            <hydrodynamics>
+                <link>base_link</link>
+                <added_mass_linear>${added_mass_linear}</added_mass_linear>
+                <added_mass_angular>${added_mass_angular}</added_mass_angular>
+                <damping_linear>${damping_linear}</damping_linear>
+                <damping_angular>${damping_angular}</damping_angular>
+            </hydrodynamics>
+        </plugin>
     </gazebo>
 </robot>

File: urdf/thruster_macro.xacro (robot description, xacro)
@@ -1,5 +1,5 @@
 <?xml version="1.0"?>
 <robot xmlns:xacro="http://www.ros.org/wiki/xacro">
-    <xacro:macro name="thruster" params="suffix parent xyz axis cw">
+    <xacro:macro name="thruster" params="suffix parent xyz axis cw color number">
         <xacro:include filename="$(find hippo_sim)/urdf/thruster_params.xacro" />
         <xacro:property name="mount_link" value="${suffix}_thruster_mount_link" />
@@ -105,4 +105,5 @@
                     <rpm_scaler>${rpm_scaler}</rpm_scaler>
                     <max_rpm>${max_rpm}</max_rpm>
+                    <thruster_number>${number}</thruster_number>
                 </thruster_config>
             </plugin>
@@ -119,5 +120,5 @@
                             <roughness>0.3</roughness>
                             <environment_map>$(find hippo_sim)/textures/env_map.dds</environment_map>
-                            <albedo_map>$(find hippo_sim)/textures/red.png</albedo_map>
+                            <albedo_map>$(find hippo_sim)/textures/${color}.png</albedo_map>
                         </metal>
                     </pbr>

File: urdf/thruster_params.xacro (robot description, xacro)
@@ -5,6 +5,6 @@
     <xacro:property name="thruster_iyy" value="1e-6" />
     <xacro:property name="thruster_izz" value="1e-6" />
-    <xacro:property name="thrust_linear_coeff" value="15.89" />
-    <xacro:property name="thrust_quadratic_coeff" value="23.2" />
+    <xacro:property name="thrust_linear_coeff" value="15.89e-2" />
+    <xacro:property name="thrust_quadratic_coeff" value="23.2e-2" />
     <xacro:property name="torque_constant" value="10.0" />
     <xacro:property name="rpm_scaler" value="10.0" />

Commit message: thruster applies torque

File: urdf/hippo2.xacro (robot description, xacro)
@@ -94,13 +94,13 @@
         </visual>
     </gazebo>
-    <xacro:thruster parent="base_link" suffix="port_top" xyz="0 -${thruster_r / 2**0.5} ${thruster_r / 2**0.5}" axis="1 0 0" cw="true" color="red" number="0" />
-    <xacro:thruster parent="base_link" suffix="starboard_top" xyz="0 ${thruster_r / 2**0.5} ${thruster_r / 2**0.5}" axis="1 0 0" cw="false" color="green" number="1" />
-    <xacro:thruster parent="base_link" suffix="starboard_bot" xyz="0 ${thruster_r / 2**0.5} -${thruster_r / 2**0.5}" axis="1 0 0" cw="true" color="grey" number="2" />
-    <xacro:thruster parent="base_link" suffix="port_bot" xyz="0 -${thruster_r / 2**0.5} -${thruster_r / 2**0.5}" axis="1 0 0" cw="false" color="grey" number="3" />
+    <xacro:thruster parent="base_link" suffix="port_top" xyz="0 ${thruster_r / 2**0.5} ${thruster_r / 2**0.5}" axis="1 0 0" turning_direction="cw" propeller_direction="cw" color="red" number="0" />
+    <xacro:thruster parent="base_link" suffix="starboard_top" xyz="0 -${thruster_r / 2**0.5} ${thruster_r / 2**0.5}" axis="1 0 0" turning_direction="cw" propeller_direction="ccw" color="green" number="1" />
+    <xacro:thruster parent="base_link" suffix="starboard_bot" xyz="0 -${thruster_r / 2**0.5} -${thruster_r / 2**0.5}" axis="1 0 0" turning_direction="cw" propeller_direction="cw" color="grey" number="2" />
+    <xacro:thruster parent="base_link" suffix="port_bot" xyz="0 ${thruster_r / 2**0.5} -${thruster_r / 2**0.5}" axis="1 0 0" turning_direction="cw" propeller_direction="ccw" color="grey" number="3" />
     <gazebo>
         <plugin filename="BuoyancyPlugin" name="ignition::gazebo::systems::BuoyancyPlugin">
             <buoyancy>
                 <link_name>base_link</link_name>
-                <origin>0 0 0.002</origin>
+                <origin>0 0 0.000</origin>
                 <force_added>0</force_added>
                 <compensation>1.01</compensation>

File: urdf/thruster_macro.xacro (robot description, xacro)
@@ -1,5 +1,5 @@
 <?xml version="1.0"?>
 <robot xmlns:xacro="http://www.ros.org/wiki/xacro">
-    <xacro:macro name="thruster" params="suffix parent xyz axis cw color number">
+    <xacro:macro name="thruster" params="suffix parent xyz axis turning_direction propeller_direction color number">
         <xacro:include filename="$(find hippo_sim)/urdf/thruster_params.xacro" />
         <xacro:property name="mount_link" value="${suffix}_thruster_mount_link" />
@@ -48,5 +48,5 @@
             <preserveFixedJoint>true</preserveFixedJoint>
         </gazebo>
-        <link name="${hull_link}">
+        <!-- <link name="${hull_link}">
             <origin xyz="0 0 0" rpy="0 0 0" />
             <inertial>
@@ -82,5 +82,5 @@
             <parent link="${parent}" />
             <child link="${hull_link}" />
-        </joint>
+        </joint> -->
         <link name="${propeller_link}">
             <origin xyz="0 0 0" rpy="0 0 0" />
@@ -106,4 +106,6 @@
                     <max_rpm>${max_rpm}</max_rpm>
                     <thruster_number>${number}</thruster_number>
+                    <turning_direction>${turning_direction}</turning_direction>
+                    <propeller_direction>${propeller_direction}</propeller_direction>
                 </thruster_config>
             </plugin>

File: urdf/thruster_params.xacro (robot description, xacro)
@@ -7,6 +7,6 @@
     <xacro:property name="thrust_linear_coeff" value="15.89e-2" />
     <xacro:property name="thrust_quadratic_coeff" value="23.2e-2" />
-    <xacro:property name="torque_constant" value="10.0" />
-    <xacro:property name="rpm_scaler" value="10.0" />
+    <xacro:property name="torque_constant" value="1e-2" />
+    <xacro:property name="rpm_scaler" value="1" />
     <xacro:property name="max_rpm" value="800" />
 </robot>

Commit message: model details

File: urdf/hippo2.xacro (robot description, xacro)
@@ -4,4 +4,7 @@
     <xacro:include filename="$(find hippo_sim)/urdf/thruster_macro.xacro" />
     <xacro:include filename="$(find hippo_sim)/urdf/hippo2_args.xacro" />
+    <xacro:include filename="$(find hippo_sim)/urdf/clamp_macro.xacro" />
+    <xacro:include filename="$(find hippo_sim)/urdf/mount_macro.xacro" />
+    <xacro:property name="thruster_xy" value="${thruster_r / 2**0.5}" />
     <gazebo>
         <static>false</static>
@@ -54,4 +57,6 @@
         <preserveFixedJoint>true</preserveFixedJoint>
     </gazebo>
+    <xacro:clamp parent="base_link" suffix="clamp_lower" xyz="0 0 0" rpy="${radians(90)} 0 0" />
+    <xacro:clamp parent="base_link" suffix="clamp_upper" xyz="0 0 0" rpy="${radians(-90)} 0 0" />
     <gazebo reference="base_link">
         <sensor name="imu_sensor" type="imu">
@@ -98,4 +103,8 @@
     <xacro:thruster parent="base_link" suffix="starboard_bot" xyz="0 -${thruster_r / 2**0.5} -${thruster_r / 2**0.5}" axis="1 0 0" turning_direction="cw" propeller_direction="cw" color="grey" number="2" />
     <xacro:thruster parent="base_link" suffix="port_bot" xyz="0 ${thruster_r / 2**0.5} -${thruster_r / 2**0.5}" axis="1 0 0" turning_direction="cw" propeller_direction="ccw" color="grey" number="3" />
+    <xacro:mount parent="base_link" suffix="port_top" xyz="0 ${thruster_r / 2**0.5} ${thruster_r / 2**0.5}" rpy="${radians(-45)} 0 0" />
+    <xacro:mount parent="base_link" suffix="starboard_top" xyz="0 -${thruster_r / 2**0.5} ${thruster_r / 2**0.5}" rpy="${radians(45)} 0 0" />
+    <xacro:mount parent="base_link" suffix="starboard_bot" xyz="0 -${thruster_r / 2**0.5} -${thruster_r / 2**0.5}" rpy="${radians(135)} 0 0" />
+    <xacro:mount parent="base_link" suffix="port_bot" xyz="0 ${thruster_r / 2**0.5} -${thruster_r / 2**0.5}" rpy="${radians(-135)} 0 0" />
     <gazebo>
         <plugin filename="BuoyancyPlugin" name="ignition::gazebo::systems::BuoyancyPlugin">

File: urdf/hippo2_params.xacro (robot description, xacro)
@@ -5,5 +5,5 @@
     <xacro:property name="iyy" value="0.010717" />
     <xacro:property name="izz" value="0.010717" />
-    <xacro:property name="thruster_r" value="0.09" />
+    <xacro:property name="thruster_r" value="0.097" />
     <xacro:property name="added_mass_linear" value="1.11 2.8 2.8" />
     <xacro:property name="added_mass_angular" value="0.00451 0.0163 0.0163"/>

File: urdf/thruster_macro.xacro (robot description, xacro)
@@ -91,5 +91,5 @@
             <visual>
                 <geometry>
-                    <mesh filename="$(find hippo_sim)/meshes/propeller.dae" />
+                    <mesh filename="$(find hippo_sim)/meshes/propeller_${propeller_direction}.dae" />
                 </geometry>
             </visual>

Commit message: camera added

File: urdf/hippo2.xacro (robot description, xacro)
@@ -6,4 +6,5 @@
     <xacro:include filename="$(find hippo_sim)/urdf/clamp_macro.xacro" />
     <xacro:include filename="$(find hippo_sim)/urdf/mount_macro.xacro" />
+    <xacro:include filename="$(find hippo_sim)/urdf/camera/camera_macro.xacro" />
     <xacro:property name="thruster_xy" value="${thruster_r / 2**0.5}" />
     <gazebo>
@@ -107,4 +108,5 @@
     <xacro:mount parent="base_link" suffix="starboard_bot" xyz="0 -${thruster_r / 2**0.5} -${thruster_r / 2**0.5}" rpy="${radians(135)} 0 0" />
     <xacro:mount parent="base_link" suffix="port_bot" xyz="0 ${thruster_r / 2**0.5} -${thruster_r / 2**0.5}" rpy="${radians(-135)} 0 0" />
+    <xacro:camera_macro parent="base_link" prefix="vertical_camera" xyz="${camera_position}" rpy="0 ${radians(90)} 0" />
     <gazebo>
         <plugin filename="ignition-gazebo-pose-publisher-system" name="ignition::gazebo::systems::PosePublisher">

File: urdf/hippo2_params.xacro (robot description, xacro)
@@ -10,3 +10,4 @@
     <xacro:property name="damping_linear" value="5.39 17.36 17.36"/>
     <xacro:property name="damping_angular" value="0.00174 0.007 0.007"/>
+    <xacro:property name="camera_position" value="-0.1, 0.0 -0.03" />
 </robot>
