Commit message: added pose plugin

File: urdf/hippo3/hippo3.xacro (robot description, xacro)
@@ -131,4 +131,8 @@
             </hydrodynamics>
         </plugin>
+        <plugin filename="PosePlugin" name="ignition::gazebo::systems::PosePlugin">
+            <link>base_link</link>
+            <update_rate>50.0</update_rate>
+        </plugin>
     </gazebo>
 </robot>
