Commit message: odometry plugin added

File: models/hippo3/urdf/hippo3.xacro (robot description, xacro)
@@ -136,4 +136,9 @@
             <base_topic>ground_truth/pose</base_topic>
         </plugin>
+        <plugin filename="OdometryPlugin" name="ignition::gazebo::systems::OdometryPlugin">
+            <link>base_link</link>
+            <update_rate>50.0</update_rate>
+            <base_topic>ground_truth/odometry</base_topic>
+        </plugin>
     </gazebo>
 </robot>
