Commit message: improved educated guess for camera position

File: models/hippo3/urdf/hippo3_params.xacro (robot description, xacro)
@@ -10,4 +10,4 @@
     <xacro:property name="damping_linear" value="5.39 17.36 17.36"/>
     <xacro:property name="damping_angular" value="0.00174 0.007 0.007"/>
-    <xacro:property name="camera_position" value="-0.1, 0.0 -0.03" />
+    <xacro:property name="camera_position" value="0.15, 0.0 -0.03" />
 </robot>
