Commit message: changed time constant to reasonable value

File: models/thruster/urdf/thruster_params.xacro (robot description, xacro)
@@ -10,5 +10,5 @@
     <xacro:property name="rpm_scaler" value="1" />
     <xacro:property name="max_rpm" value="800" />
-    <xacro:property name="timeconstant_up" value="1.0" />
-    <xacro:property name="timeconstant_down" value="1.0" />
+    <xacro:property name="timeconstant_up" value="0.05" />
+    <xacro:property name="timeconstant_down" value="0.05" />
 </robot>
