Commit message: added changes by niklastkl

File: models/thruster/urdf/t200_params.xacro (robot description, xacro)
@@ -7,5 +7,5 @@
     <!-- based on 14V performance data and forced interception at 0.0 -->
     <xacro:property name="thrust_quadratic_coeff" value="0.015547" />
-    <xacro:property name="thrust_linear_coeff" value="0.04243" />
+    <xacro:property name="thrust_linear_coeff" value="-0.04243" />
     <xacro:property name="thrust_constant_coeff" value="0.0" />
     <xacro:property name="torque_constant" value="0.0" />

Commit message: change t200 linear thrust coefficient to zero to avoid accidental deadzone for very small thrusts

File: models/thruster/urdf/t200_params.xacro (robot description, xacro)
@@ -7,5 +7,7 @@
     <!-- based on 14V performance data and forced interception at 0.0 -->
     <xacro:property name="thrust_quadratic_coeff" value="0.015547" />
-    <xacro:property name="thrust_linear_coeff" value="-0.04243" />
+    <!-- Niklas value for thrust_linear_coeff: -0.04243-->
+    <!-- changed to 0.0 to avoid accidental deadzone since very small rotational velocities lead to negative thrusts which get set to zero -->
+    <xacro:property name="thrust_linear_coeff" value="0.0" />
     <xacro:property name="thrust_constant_coeff" value="0.0" />
     <xacro:property name="torque_constant" value="0.0" />
