Commit message: created bluerof urdf as macro, modified buoyancy plugin as parameters are not loaded properly

File: models/bluerov/urdf/bluerov.xacro (robot description, xacro)
@@ -1,90 +1,7 @@
 <?xml version="1.0"?>
 <robot xmlns:xacro="http://www.ros.org/wiki/xacro" name="hippocampus">
-    <xacro:include filename="$(find hippo_sim)/models/bluerov/urdf/bluerov_params.xacro" />
-    <xacro:include filename="$(find hippo_sim)/models/thruster/urdf/thruster_macro.xacro" />
-    <xacro:include filename="$(find hippo_sim)/models/hippo3/urdf/mount_macro.xacro" />
-    <xacro:include filename="$(find hippo_sim)/models/hippo3/urdf/clamp_macro.xacro" />
-    <!-- <xacro:include filename="$(find hippo_sim)/models/range_sensor/urdf/range_sensor_macro.xacro" />
-    <xacro:include filename="$(find hippo_sim)/models/camera/urdf/camera_macro.xacro" /> -->
-    <xacro:property name="thruster_xy" value="${thruster_r / 2**0.5}" /><gazebo>
-        <static>false</static>
-    </gazebo>
-    <link name="base_link">
-        <inertial name="base_link_inertial">
-            <mass value="${base_mass}" />
-            <inertia ixx="${ixx}" ixy="0.0" ixz="0.0" iyy="${iyy}" iyz="0.0" izz="${izz}" />
-        </inertial>
-        <visual name="base_link_visual">
-            <geometry>
-                <mesh filename="$(find hippo_sim)/models/bluerov/meshes/bluerov.dae" />
-            </geometry>
-        </visual>
-    </link>
-    <xacro:thruster parent="base_link" model="t200" suffix="front_starboard_horizontal" xyz="0.14 -0.10 0" rpy="0 0 ${radians(45)}" turning_direction="cw" propeller_direction="ccw" color="red" number="0" />
-    <xacro:thruster parent="base_link" model="t200" suffix="front_port_horizontal" xyz="0.14 0.10 0" rpy="0 0 ${radians(-45)}" turning_direction="cw" propeller_direction="ccw" color="green" number="1" />
-    <xacro:thruster parent="base_link" model="t200" suffix="rear_starboard_horizontal" xyz="-0.14 -0.10 0" rpy="0 0 ${radians(135)}" turning_direction="cw" propeller_direction="cw" color="grey" number="2" />
-    <xacro:thruster parent="base_link" model="t200" suffix="rear_port_horizontal" xyz="-0.14 0.10 0" rpy="0 0 ${radians(-135)}" turning_direction="cw" propeller_direction="cw" color="grey" number="3" />
-    <xacro:thruster parent="base_link" model="t200" suffix="front_starboard_vertical" xyz="0.12 -0.22 0.06" rpy="0 ${radians(-90)} 0" turning_direction="cw" propeller_direction="ccw" color="red" number="4" />
-    <xacro:thruster parent="base_link" model="t200" suffix="front_port_vertical" xyz="0.12 0.22 0.06" rpy="0 ${radians(-90)} 0" turning_direction="ccw" propeller_direction="ccw" color="green" number="5" />
-    <xacro:thruster parent="base_link" model="t200" suffix="rear_starboard_vertical" xyz="-0.12 -0.22 0.06" rpy="0 ${radians(-90)} 0" turning_direction="ccw" propeller_direction="ccw" color="grey" number="6" />
-    <xacro:thruster parent="base_link" model="t200" suffix="rear_port_vertical" xyz="-0.12 0.22 0.06" rpy="0 ${radians(-90)} 0" turning_direction="cw" propeller_direction="ccw" color="grey" number="7" />
-    <gazebo>
-        <plugin filename="buoyancy" name="hippo_gz_plugins::buoyancy">
-            <buoyancy>
-                <link_name>base_link</link_name>
-                <origin>0 0 0.01</origin>
-                <force_added>0</force_added>
-                <compensation>1.01</compensation>
-                <height_scale_limit>0.1</height_scale_limit>
-            </buoyancy>
-        </plugin>
-        <plugin filename="hydrodynamics" name="hippo_gz_plugins::hydrodynamics">
-            <hydrodynamics>
-                <link>base_link</link>
-                <added_mass_linear>${added_mass_linear}</added_mass_linear>
-                <added_mass_angular>${added_mass_angular}</added_mass_angular>
-                <damping_linear>${damping_linear}</damping_linear>
-                <damping_angular>${damping_angular}</damping_angular>
-            </hydrodynamics>
-        </plugin>
-        <plugin filename="pose" name="hippo_gz_plugins::pose">
-            <link>base_link</link>
-            <update_rate>50.0</update_rate>
-            <base_topic>ground_truth/pose</base_topic>
-        </plugin>
-        <plugin filename="odometry" name="hippo_gz_plugins::odometry">
-            <link>base_link</link>
-            <update_rate>50.0</update_rate>
-            <base_topic>ground_truth/odometry</base_topic>
-        </plugin>
-        <plugin filename="barometer" name="hippo_gz_plugins::barometer">
-            <link>base_link</link>
-            <update_rate>100.0</update_rate>
-            <base_topic>pressure</base_topic>
-            <atmospheric_pressure>101325.0</atmospheric_pressure>
-            <water_surface_offset>0.0</water_surface_offset>
-            <position>-0.15 0 0</position>
-        </plugin>
-        <plugin filename="range_sensor" name="hippo_gz_plugins::range_sensor">
-            <link>base_link</link>
-            <range_topic>range_topic</range_topic>
-            <update_rate>20.0</update_rate>
-            <model name="range_tag_00">
-                <link>base_link</link>
-                <id>0</id>
-            </model>
-            <model name="range_tag_01">
-                <link>base_link</link>
-                <id>1</id>
-            </model>
-            <model name="range_tag_02">
-                <link>base_link</link>
-                <id>2</id>
-            </model>
-            <model name="range_tag_03">
-                <link>base_link</link>
-                <id>3</id>
-            </model>
-        </plugin>
-    </gazebo>
+    <xacro:arg name="base_link_name" default="base_link"/>
+    <xacro:include filename="$(find hippo_sim)/models/bluerov/urdf/bluerov_macro.xacro"/>
+    <xacro:bluerov base_link_name="$(arg base_link_name)">
+    </xacro:bluerov>
 </robot>

File: models/bluerov/urdf/bluerov_params.xacro (robot description, xacro)
@@ -9,6 +9,7 @@
     <xacro:property name="damping_linear" value="7 7 7" />
     <xacro:property name="damping_angular" value="0.3 0.3 0.3" />
-    <xacro:property name="buoyancy_compensation" value="1.001" />
-    <xacro:property name="buoyancy_origin" value="0 0 0.005" />
+    <!-- alpha manipulator weight underwater: 1.272 kg - 0.5719 kg = 0.7001  => 0.7001 / 11.0 (mass bluerov) = 0.064-->
+    <xacro:property name="buoyancy_compensation" value="1.065" /> <!--1.001 default -->
+    <xacro:property name="buoyancy_origin" value="0 0 0.05" />
     <xacro:property name="barometer_position" value="-0.15 0 -0.05" />
     <xacro:property name="barometer_noise" value="100.0" />

Commit message: adapted changes in namespace and clock after merge

File: models/bluerov/urdf/bluerov.xacro (robot description, xacro)
@@ -3,5 +3,5 @@
     <xacro:arg name="base_link_name" default="base_link"/>
     <xacro:include filename="$(find hippo_sim)/models/bluerov/urdf/bluerov_macro.xacro"/>
-    <xacro:bluerov base_link_name="$(arg base_link_name)">
+    <xacro:bluerov base_link_name="$(arg base_link_name)" link_ns="$(arg vehicle_name)/">
     </xacro:bluerov>
 </robot>

File: models/bluerov/urdf/bluerov_macro.xacro (robot description, xacro)
@@ -1,5 +1,5 @@
 <?xml version="1.0"?>
 <robot xmlns:xacro="http://www.ros.org/wiki/xacro" name="hippocampus">
-    <xacro:macro name="bluerov" params="base_link_name:=base_link use_uvms_param:=False rviz_model:=False simulate_kinematics:=False">
+    <xacro:macro name="bluerov" params="base_link_name:=base_link link_ns use_uvms_param:=False rviz_model:=False simulate_kinematics:=False">
         <xacro:if value="${use_uvms_param == True}">
             <xacro:include filename="$(find hippo_sim)/models/bluerov/urdf/bluerov_params_uvms.xacro" />
@@ -16,5 +16,5 @@
             <static>false</static>
         </gazebo>
-        <link name="${base_link_name}">
+        <link name="${link_ns}${base_link_name}">
             <xacro:unless value="${rviz_model == True}">
             <inertial name="base_link_inertial">
@@ -30,21 +30,21 @@
         </link>
         <xacro:unless value="${rviz_model == True}">
-            <xacro:thruster parent="${base_link_name}" model="t200" suffix="front_starboard_horizontal" xyz="0.14 -0.10 0" rpy="0 0 ${radians(45)}" turning_direction="cw" propeller_direction="ccw" color="red" number="0"/>
-            <xacro:thruster parent="${base_link_name}" model="t200" suffix="front_port_horizontal" xyz="0.14 0.10 0" rpy="0 0 ${radians(-45)}" turning_direction="cw" propeller_direction="ccw" color="green" number="1" />
-            <xacro:thruster parent="${base_link_name}" model="t200" suffix="rear_starboard_horizontal" xyz="-0.14 -0.10 0" rpy="0 0 ${radians(135)}" turning_direction="cw" propeller_direction="cw" color="grey" number="2" />
-            <xacro:thruster parent="${base_link_name}" model="t200" suffix="rear_port_horizontal" xyz="-0.14 0.10 0" rpy="0 0 ${radians(-135)}" turning_direction="cw" propeller_direction="cw" color="grey" number="3" />
-            <xacro:thruster parent="${base_link_name}" model="t200" suffix="front_starboard_vertical" xyz="0.12 -0.22 0.06" rpy="0 ${radians(-90)} 0" turning_direction="cw" propeller_direction="ccw" color="red" number="4" />
-            <xacro:thruster parent="${base_link_name}" model="t200" suffix="front_port_vertical" xyz="0.12 0.22 0.06" rpy="0 ${radians(-90)} 0" turning_direction="ccw" propeller_direction="ccw" color="green" number="5" />
-            <xacro:thruster parent="${base_link_name}" model="t200" suffix="rear_starboard_vertical" xyz="-0.12 -0.22 0.06" rpy="0 ${radians(-90)} 0" turning_direction="ccw" propeller_direction="ccw" color="grey" number="6" />
-            <xacro:thruster parent="${base_link_name}" model="t200" suffix="rear_port_vertical" xyz="-0.12 0.22 0.06" rpy="0 ${radians(-90)} 0" turning_direction="cw" propeller_direction="ccw" color="grey" number="7" />
+            <xacro:thruster parent="${link_ns}${base_link_name}" model="t200" suffix="front_starboard_horizontal" xyz="0.14 -0.10 0" rpy="0 0 ${radians(45)}" turning_direction="cw" propeller_direction="ccw" color="red" number="0"/>
+            <xacro:thruster parent="${link_ns}${base_link_name}" model="t200" suffix="front_port_horizontal" xyz="0.14 0.10 0" rpy="0 0 ${radians(-45)}" turning_direction="cw" propeller_direction="ccw" color="green" number="1" />
+            <xacro:thruster parent="${link_ns}${base_link_name}" model="t200" suffix="rear_starboard_horizontal" xyz="-0.14 -0.10 0" rpy="0 0 ${radians(135)}" turning_direction="cw" propeller_direction="cw" color="grey" number="2" />
+            <xacro:thruster parent="${link_ns}${base_link_name}" model="t200" suffix="rear_port_horizontal" xyz="-0.14 0.10 0" rpy="0 0 ${radians(-135)}" turning_direction="cw" propeller_direction="cw" color="grey" number="3" />
+            <xacro:thruster parent="${link_ns}${base_link_name}" model="t200" suffix="front_starboard_vertical" xyz="0.12 -0.22 0.06" rpy="0 ${radians(-90)} 0" turning_direction="cw" propeller_direction="ccw" color="red" number="4" />
+            <xacro:thruster parent="${link_ns}${base_link_name}" model="t200" suffix="front_port_vertical" xyz="0.12 0.22 0.06" rpy="0 ${radians(-90)} 0" turning_direction="ccw" propeller_direction="ccw" color="green" number="5" />
+            <xacro:thruster parent="${link_ns}${base_link_name}" model="t200" suffix="rear_starboard_vertical" xyz="-0.12 -0.22 0.06" rpy="0 ${radians(-90)} 0" turning_direction="ccw" propeller_direction="ccw" color="grey" number="6" />
+            <xacro:thruster parent="${link_ns}${base_link_name}" model="t200" suffix="rear_port_vertical" xyz="-0.12 0.22 0.06" rpy="0 ${radians(-90)} 0" turning_direction="cw" propeller_direction="ccw" color="grey" number="7" />
         </xacro:unless>
         <gazebo>
             <xacro:if value="${simulate_kinematics == True}">
                 <plugin filename="kinematic_control" name="hippo_gz_plugins::kinematic_control">
-                    <link_name>${base_link_name}</link_name>
+                    <link_name>${link_ns}${base_link_name}</link_name>
                 </plugin>
                 <!--
                 <plugin name="ignition::gazebo::systems::VelocityControl" filename="ignition-gazebo-velocity-control-system">
-                    <link_name>${base_link_name}</link_name>
+                    <link_name>${link_ns}${base_link_name}</link_name>
                 </plugin>
                 -->
@@ -53,5 +53,5 @@
                 <plugin filename="buoyancy" name="hippo_gz_plugins::buoyancy">
                     <buoyancy>
-                        <link_name>${base_link_name}</link_name>
+                        <link_name>${link_ns}${base_link_name}</link_name>
                         <origin>${buoyancy_origin}</origin>
                         <force_added>0</force_added>
@@ -62,5 +62,5 @@
                 <plugin filename="hydrodynamics" name="hippo_gz_plugins::hydrodynamics">
                     <hydrodynamics>
-                        <link>${base_link_name}</link>
+                        <link>${link_ns}${base_link_name}</link>
                         <added_mass_linear>${added_mass_linear}</added_mass_linear>
                         <added_mass_angular>${added_mass_angular}</added_mass_angular>
@@ -71,10 +71,10 @@
             </xacro:unless>
             <plugin filename="pose" name="hippo_gz_plugins::pose">
-                <link>${base_link_name}</link>
+                <link>${link_ns}${base_link_name}</link>
                 <update_rate>50.0</update_rate>
                 <base_topic>ground_truth/pose</base_topic>
             </plugin>
             <plugin filename="odometry" name="hippo_gz_plugins::odometry">
-                <link>${base_link_name}</link>
+                <link>${link_ns}${base_link_name}</link>
                 <update_rate>50.0</update_rate>
                 <base_topic>ground_truth/odometry</base_topic>
@@ -82,5 +82,5 @@
             <!--
             <plugin filename="barometer" name="hippo_gz_plugins::barometer">
-                <link>${base_link_name}</link>
+                <link>${link_ns}${base_link_name}</link>
                 <update_rate>100.0</update_rate>
                 <base_topic>pressure</base_topic>
@@ -90,21 +90,21 @@
             </plugin>
             <plugin filename="range_sensor" name="hippo_gz_plugins::range_sensor">
-                <link>${base_link_name}</link>
+                <link>${link_ns}${base_link_name}</link>
                 <range_topic>range_topic</range_topic>
                 <update_rate>20.0</update_rate>
                 <model name="range_tag_00">
-                    <link>${base_link_name}</link>
+                    <link>${link_ns}${base_link_name}</link>
                     <id>0</id>
                 </model>
                 <model name="range_tag_01">
-                    <link>${base_link_name}</link>
+                    <link>${link_ns}${base_link_name}</link>
                     <id>1</id>
                 </model>
                 <model name="range_tag_02">
-                    <link>${base_link_name}</link>
+                    <link>${link_ns}${base_link_name}</link>
                     <id>2</id>
                 </model>
                 <model name="range_tag_03">
-                    <link>${base_link_name}</link>
+                    <link>${link_ns}${base_link_name}</link>
                     <id>3</id>
                 </model>

File: models/bluerov/urdf/bluerov_rviz.xacro (robot description, xacro)
@@ -3,5 +3,5 @@
     <xacro:arg name="base_link_name" default="base_link"/>
     <xacro:include filename="$(find hippo_sim)/models/bluerov/urdf/bluerov_macro.xacro"/>
-    <xacro:bluerov base_link_name="$(arg base_link_name)" rviz_model="True">
+    <xacro:bluerov base_link_name="$(arg base_link_name)" link_ns="$(arg vehicle_name)/" rviz_model="True">
     </xacro:bluerov>
 </robot>

Commit message: revert to upstream status

File: models/bluerov/urdf/bluerov.xacro (robot description, xacro)
@@ -1,8 +1,90 @@
 <?xml version="1.0"?>
 <robot xmlns:xacro="http://www.ros.org/wiki/xacro" name="hippocampus">
-    <xacro:arg name="base_link_name" default="base_link"/>
-    <xacro:arg name="vehicle_name" default="bluerov"/>
-    <xacro:include filename="$(find hippo_sim)/models/bluerov/urdf/bluerov_macro.xacro"/>
-    <xacro:bluerov base_link_name="$(arg base_link_name)" link_ns="$(arg vehicle_name)/">
-    </xacro:bluerov>
+    <xacro:include filename="$(find hippo_sim)/models/bluerov/urdf/bluerov_params.xacro" />
+    <xacro:include filename="$(find hippo_sim)/models/thruster/urdf/thruster_macro.xacro" />
+    <xacro:include filename="$(find hippo_sim)/models/hippo3/urdf/mount_macro.xacro" />
+    <xacro:include filename="$(find hippo_sim)/models/hippo3/urdf/clamp_macro.xacro" />
+    <!-- <xacro:include filename="$(find hippo_sim)/models/range_sensor/urdf/range_sensor_macro.xacro" />
+    <xacro:include filename="$(find hippo_sim)/models/camera/urdf/camera_macro.xacro" /> -->
+    <xacro:property name="thruster_xy" value="${thruster_r / 2**0.5}" /><gazebo>
+        <static>false</static>
+    </gazebo>
+    <link name="base_link">
+        <inertial name="base_link_inertial">
+            <mass value="${base_mass}" />
+            <inertia ixx="${ixx}" ixy="0.0" ixz="0.0" iyy="${iyy}" iyz="0.0" izz="${izz}" />
+        </inertial>
+        <visual name="base_link_visual">
+            <geometry>
+                <mesh filename="$(find hippo_sim)/models/bluerov/meshes/bluerov.dae" />
+            </geometry>
+        </visual>
+    </link>
+    <xacro:thruster parent="base_link" model="t200" suffix="front_starboard_horizontal" xyz="0.14 -0.10 0" rpy="0 0 ${radians(45)}" turning_direction="cw" propeller_direction="ccw" color="red" number="0" />
+    <xacro:thruster parent="base_link" model="t200" suffix="front_port_horizontal" xyz="0.14 0.10 0" rpy="0 0 ${radians(-45)}" turning_direction="cw" propeller_direction="ccw" color="green" number="1" />
+    <xacro:thruster parent="base_link" model="t200" suffix="rear_starboard_horizontal" xyz="-0.14 -0.10 0" rpy="0 0 ${radians(135)}" turning_direction="cw" propeller_direction="cw" color="grey" number="2" />
+    <xacro:thruster parent="base_link" model="t200" suffix="rear_port_horizontal" xyz="-0.14 0.10 0" rpy="0 0 ${radians(-135)}" turning_direction="cw" propeller_direction="cw" color="grey" number="3" />
+    <xacro:thruster parent="base_link" model="t200" suffix="front_starboard_vertical" xyz="0.12 -0.22 0.06" rpy="0 ${radians(-90)} 0" turning_direction="cw" propeller_direction="ccw" color="red" number="4" />
+    <xacro:thruster parent="base_link" model="t200" suffix="front_port_vertical" xyz="0.12 0.22 0.06" rpy="0 ${radians(-90)} 0" turning_direction="ccw" propeller_direction="ccw" color="green" number="5" />
+    <xacro:thruster parent="base_link" model="t200" suffix="rear_starboard_vertical" xyz="-0.12 -0.22 0.06" rpy="0 ${radians(-90)} 0" turning_direction="ccw" propeller_direction="ccw" color="grey" number="6" />
+    <xacro:thruster parent="base_link" model="t200" suffix="rear_port_vertical" xyz="-0.12 0.22 0.06" rpy="0 ${radians(-90)} 0" turning_direction="cw" propeller_direction="ccw" color="grey" number="7" />
+    <gazebo>
+        <plugin filename="buoyancy" name="hippo_gz_plugins::buoyancy">
+            <buoyancy>
+                <link_name>base_link</link_name>
+                <origin>0 0 0.01</origin>
+                <force_added>0</force_added>
+                <compensation>1.01</compensation>
+                <height_scale_limit>0.1</height_scale_limit>
+            </buoyancy>
+        </plugin>
+        <plugin filename="hydrodynamics" name="hippo_gz_plugins::hydrodynamics">
+            <hydrodynamics>
+                <link>base_link</link>
+                <added_mass_linear>${added_mass_linear}</added_mass_linear>
+                <added_mass_angular>${added_mass_angular}</added_mass_angular>
+                <damping_linear>${damping_linear}</damping_linear>
+                <damping_angular>${damping_angular}</damping_angular>
+            </hydrodynamics>
+        </plugin>
+        <plugin filename="pose" name="hippo_gz_plugins::pose">
+            <link>base_link</link>
+            <update_rate>50.0</update_rate>
+            <base_topic>ground_truth/pose</base_topic>
+        </plugin>
+        <plugin filename="odometry" name="hippo_gz_plugins::odometry">
+            <link>base_link</link>
+            <update_rate>50.0</update_rate>
+            <base_topic>ground_truth/odometry</base_topic>
+        </plugin>
+        <plugin filename="barometer" name="hippo_gz_plugins::barometer">
+            <link>base_link</link>
+            <update_rate>100.0</update_rate>
+            <base_topic>pressure</base_topic>
+            <atmospheric_pressure>101325.0</atmospheric_pressure>
+            <water_surface_offset>0.0</water_surface_offset>
+            <position>-0.15 0 0</position>
+        </plugin>
+        <plugin filename="range_sensor" name="hippo_gz_plugins::range_sensor">
+            <link>base_link</link>
+            <range_topic>range_topic</range_topic>
+            <update_rate>20.0</update_rate>
+            <model name="range_tag_00">
+                <link>base_link</link>
+                <id>0</id>
+            </model>
+            <model name="range_tag_01">
+                <link>base_link</link>
+                <id>1</id>
+            </model>
+            <model name="range_tag_02">
+                <link>base_link</link>
+                <id>2</id>
+            </model>
+            <model name="range_tag_03">
+                <link>base_link</link>
+                <id>3</id>
+            </model>
+        </plugin>
+    </gazebo>
 </robot>

File: models/thruster/urdf/t200_params.xacro (robot description, xacro)
@@ -12,6 +12,6 @@
     <!-- for reversed direction:  0.01268 -0.05067 0.0 -->
     <!-- Throttle = f(revs/s) -->
-    <xacro:property name="velocity_quadratic_coeff" value="0.00914"/>
-    <xacro:property name="velocity_linear_coeff" value="-0.2228"/>
+    <xacro:property name="velocity_quadratic_coeff" value="1.2679e-4"/>
+    <xacro:property name="velocity_linear_coeff" value="1.1105e-2"/>
     <xacro:property name="velocity_constant_coeff" value="0.0"/>
     <xacro:property name="rpm_scaler" value="10" />
