Commit message: revert to upstream

File: models/bluerov/urdf/bluerov.xacro (robot description, xacro)
@@ -1,7 +1,90 @@
 <?xml version="1.0"?>
 <robot xmlns:xacro="http://www.ros.org/wiki/xacro" name="hippocampus">
-    <xacro:arg name="base_link_name" default="base_link"/>
-    <xacro:include filename="$(find hippo_sim)/models/bluerov/urdf/bluerov_macro.xacro"/>
-    <xacro:bluerov base_link_name="$(arg base_link_name)">
-    </xacro:bluerov>
+    <xacro:include filename="$(find hippo_sim)/models/bluerov/urdf/bluerov_params.xacro" />
+    <xacro:include filename="$(find hippo_sim)/models/thruster/urdf/thruster_macro.xacro" />
+    <xacro:include filename="$(find hippo_sim)/models/hippo3/urdf/mount_macro.xacro" />
+    <xacro:bluerov base_link_name="$(arg base_link_name)" link_ns="$(arg vehicle_name)/">
+    <!-- <xacro:include filename="$(find hippo_sim)/models/range_sensor/urdf/range_sensor_macro.xacro" />
+    <xacro:include filename="$(find hippo_sim)/models/camera/urdf/camera_macro.xacro" /> -->
+    <xacro:property name="thruster_xy" value="${thruster_r / 2**0.5}" /><gazebo>
+        <static>false</static>
+    </gazebo>
+    <link name="base_link">
+        <inertial name="base_link_inertial">
+            <mass value="${base_mass}" />
+            <inertia ixx="${ixx}" ixy="0.0" ixz="0.0" iyy="${iyy}" iyz="0.0" izz="${izz}" />
+        </inertial>
+        <visual name="base_link_visual">
+            <geometry>
+                <mesh filename="$(find hippo_sim)/models/bluerov/meshes/bluerov.dae" />
+            </geometry>
+        </visual>
+    </link>
+    <xacro:thruster parent="base_link" model="t200" suffix="front_starboard_horizontal" xyz="0.14 -0.10 0" rpy="0 0 ${radians(45)}" turning_direction="cw" propeller_direction="ccw" color="red" number="0" />
+    <xacro:thruster parent="base_link" model="t200" suffix="front_port_horizontal" xyz="0.14 0.10 0" rpy="0 0 ${radians(-45)}" turning_direction="cw" propeller_direction="ccw" color="green" number="1" />
+    <xacro:thruster parent="base_link" model="t200" suffix="rear_starboard_horizontal" xyz="-0.14 -0.10 0" rpy="0 0 ${radians(135)}" turning_direction="cw" propeller_direction="cw" color="grey" number="2" />
+    <xacro:thruster parent="base_link" model="t200" suffix="rear_port_horizontal" xyz="-0.14 0.10 0" rpy="0 0 ${radians(-135)}" turning_direction="cw" propeller_direction="cw" color="grey" number="3" />
+    <xacro:thruster parent="base_link" model="t200" suffix="front_starboard_vertical" xyz="0.12 -0.22 0.06" rpy="0 ${radians(-90)} 0" turning_direction="cw" propeller_direction="ccw" color="red" number="4" />
+    <xacro:thruster parent="base_link" model="t200" suffix="front_port_vertical" xyz="0.12 0.22 0.06" rpy="0 ${radians(-90)} 0" turning_direction="ccw" propeller_direction="ccw" color="green" number="5" />
+    <xacro:thruster parent="base_link" model="t200" suffix="rear_starboard_vertical" xyz="-0.12 -0.22 0.06" rpy="0 ${radians(-90)} 0" turning_direction="ccw" propeller_direction="ccw" color="grey" number="6" />
+    <xacro:thruster parent="base_link" model="t200" suffix="rear_port_vertical" xyz="-0.12 0.22 0.06" rpy="0 ${radians(-90)} 0" turning_direction="cw" propeller_direction="ccw" color="grey" number="7" />
+    <gazebo>
+        <plugin filename="buoyancy" name="hippo_gz_plugins::buoyancy">
+            <buoyancy>
+                <link_name>base_link</link_name>
+                <origin>0 0 0.01</origin>
+                <force_added>0</force_added>
+                <compensation>1.01</compensation>
+                <height_scale_limit>0.1</height_scale_limit>
+            </buoyancy>
+        </plugin>
+        <plugin filename="hydrodynamics" name="hippo_gz_plugins::hydrodynamics">
+            <hydrodynamics>
+                <link>base_link</link>
+                <added_mass_linear>${added_mass_linear}</added_mass_linear>
+                <added_mass_angular>${added_mass_angular}</added_mass_angular>
+                <damping_linear>${damping_linear}</damping_linear>
+                <damping_angular>${damping_angular}</damping_angular>
+            </hydrodynamics>
+        </plugin>
+        <plugin filename="pose" name="hippo_gz_plugins::pose">
+            <link>base_link</link>
+            <update_rate>50.0</update_rate>
+            <base_topic>ground_truth/pose</base_topic>
+        </plugin>
+        <plugin filename="odometry" name="hippo_gz_plugins::odometry">
+            <link>base_link</link>
+            <update_rate>50.0</update_rate>
+            <base_topic>ground_truth/odometry</base_topic>
+        </plugin>
+        <plugin filename="barometer" name="hippo_gz_plugins::barometer">
+            <link>base_link</link>
+            <update_rate>100.0</update_rate>
+            <base_topic>pressure</base_topic>
+            <atmospheric_pressure>101325.0</atmospheric_pressure>
+            <water_surface_offset>0.0</water_surface_offset>
+            <position>-0.15 0 0</position>
+        </plugin>
+        <plugin filename="range_sensor" name="hippo_gz_plugins::range_sensor">
+            <link>base_link</link>
+            <range_topic>range_topic</range_topic>
+            <update_rate>20.0</update_rate>
+            <model name="range_tag_00">
+                <link>base_link</link>
+                <id>0</id>
+            </model>
+            <model name="range_tag_01">
+                <link>base_link</link>
+                <id>1</id>
+            </model>
+            <model name="range_tag_02">
+                <link>base_link</link>
+                <id>2</id>
+            </model>
+            <model name="range_tag_03">
+                <link>base_link</link>
+                <id>3</id>
+            </model>
+        </plugin>
+    </gazebo>
 </robot>

Commit message: make usage of range sensor togglable

File: models/bluerov/urdf/bluerov.xacro (robot description, xacro)
@@ -66,25 +66,27 @@
             <position>-0.15 0 0</position>
         </plugin>
-        <plugin filename="range_sensor" name="hippo_gz_plugins::range_sensor">
-            <link>base_link</link>
-            <range_topic>range_topic</range_topic>
-            <update_rate>20.0</update_rate>
-            <model name="range_tag_00">
+        <xacro:if value="$(arg use_range_sensor)">
+            <plugin filename="range_sensor" name="hippo_gz_plugins::range_sensor">
                 <link>base_link</link>
-                <id>0</id>
-            </model>
-            <model name="range_tag_01">
-                <link>base_link</link>
-                <id>1</id>
-            </model>
-            <model name="range_tag_02">
-                <link>base_link</link>
-                <id>2</id>
-            </model>
-            <model name="range_tag_03">
-                <link>base_link</link>
-                <id>3</id>
-            </model>
-        </plugin>
+                <range_topic>range_topic</range_topic>
+                <update_rate>20.0</update_rate>
+                <model name="range_tag_00">
+                    <link>base_link</link>
+                    <id>0</id>
+                </model>
+                <model name="range_tag_01">
+                    <link>base_link</link>
+                    <id>1</id>
+                </model>
+                <model name="range_tag_02">
+                    <link>base_link</link>
+                    <id>2</id>
+                </model>
+                <model name="range_tag_03">
+                    <link>base_link</link>
+                    <id>3</id>
+                </model>
+            </plugin>
+        </xacro:if>
     </gazebo>
 </robot>

File: models/bluerov/urdf/bluerov_params.xacro (robot description, xacro)
@@ -27,3 +27,4 @@
     <xacro:property name="front_camera_orientation" value="0 0 0" />
     <xacro:property name="thruster_r" value="0.097" />
+    <xacro:arg name="use_range_sensor" default="false" />
 </robot>

Commit message: make cameras configurable during launch

File: models/bluerov/urdf/bluerov.xacro (robot description, xacro)
@@ -5,7 +5,9 @@
     <xacro:include filename="$(find hippo_sim)/models/hippo3/urdf/mount_macro.xacro" />
     <xacro:include filename="$(find hippo_sim)/models/hippo3/urdf/clamp_macro.xacro" />
-    <!-- <xacro:include filename="$(find hippo_sim)/models/range_sensor/urdf/range_sensor_macro.xacro" />
-    <xacro:include filename="$(find hippo_sim)/models/camera/urdf/camera_macro.xacro" /> -->
-    <xacro:property name="thruster_xy" value="${thruster_r / 2**0.5}" /><gazebo>
+    <!-- <xacro:include filename="$(find
+    hippo_sim)/models/range_sensor/urdf/range_sensor_macro.xacro" /> -->
+    <xacro:include filename="$(find hippo_sim)/models/camera/urdf/camera_macro.xacro" />
+    <xacro:property name="thruster_xy" value="${thruster_r / 2**0.5}" />
+    <gazebo>
         <static>false</static>
     </gazebo>
@@ -21,12 +23,38 @@
         </visual>
     </link>
-    <xacro:thruster parent="base_link" model="t200" suffix="front_starboard_horizontal" xyz="0.14 -0.10 0" rpy="0 0 ${radians(45)}" turning_direction="cw" propeller_direction="ccw" color="red" number="0" />
-    <xacro:thruster parent="base_link" model="t200" suffix="front_port_horizontal" xyz="0.14 0.10 0" rpy="0 0 ${radians(-45)}" turning_direction="cw" propeller_direction="ccw" color="green" number="1" />
-    <xacro:thruster parent="base_link" model="t200" suffix="rear_starboard_horizontal" xyz="-0.14 -0.10 0" rpy="0 0 ${radians(135)}" turning_direction="cw" propeller_direction="cw" color="grey" number="2" />
-    <xacro:thruster parent="base_link" model="t200" suffix="rear_port_horizontal" xyz="-0.14 0.10 0" rpy="0 0 ${radians(-135)}" turning_direction="cw" propeller_direction="cw" color="grey" number="3" />
-    <xacro:thruster parent="base_link" model="t200" suffix="front_starboard_vertical" xyz="0.12 -0.22 0.06" rpy="0 ${radians(-90)} 0" turning_direction="cw" propeller_direction="ccw" color="red" number="4" />
-    <xacro:thruster parent="base_link" model="t200" suffix="front_port_vertical" xyz="0.12 0.22 0.06" rpy="0 ${radians(-90)} 0" turning_direction="ccw" propeller_direction="ccw" color="green" number="5" />
-    <xacro:thruster parent="base_link" model="t200" suffix="rear_starboard_vertical" xyz="-0.12 -0.22 0.06" rpy="0 ${radians(-90)} 0" turning_direction="ccw" propeller_direction="ccw" color="grey" number="6" />
-    <xacro:thruster parent="base_link" model="t200" suffix="rear_port_vertical" xyz="-0.12 0.22 0.06" rpy="0 ${radians(-90)} 0" turning_direction="cw" propeller_direction="ccw" color="grey" number="7" />
+    <xacro:thruster parent="base_link" model="t200" suffix="front_starboard_horizontal"
+        xyz="0.14 -0.10 0" rpy="0 0 ${radians(45)}" turning_direction="cw" propeller_direction="ccw"
+        color="red" number="0" />
+    <xacro:thruster parent="base_link" model="t200" suffix="front_port_horizontal" xyz="0.14 0.10 0"
+        rpy="0 0 ${radians(-45)}" turning_direction="cw" propeller_direction="ccw" color="green"
+        number="1" />
+    <xacro:thruster parent="base_link" model="t200" suffix="rear_starboard_horizontal"
+        xyz="-0.14 -0.10 0" rpy="0 0 ${radians(135)}" turning_direction="cw"
+        propeller_direction="cw" color="grey" number="2" />
+    <xacro:thruster parent="base_link" model="t200" suffix="rear_port_horizontal" xyz="-0.14 0.10 0"
+        rpy="0 0 ${radians(-135)}" turning_direction="cw" propeller_direction="cw" color="grey"
+        number="3" />
+    <xacro:thruster parent="base_link" model="t200" suffix="front_starboard_vertical"
+        xyz="0.12 -0.22 0.06" rpy="0 ${radians(-90)} 0" turning_direction="cw"
+        propeller_direction="ccw" color="red" number="4" />
+    <xacro:thruster parent="base_link" model="t200" suffix="front_port_vertical"
+        xyz="0.12 0.22 0.06" rpy="0 ${radians(-90)} 0" turning_direction="ccw"
+        propeller_direction="ccw" color="green" number="5" />
+    <xacro:thruster parent="base_link" model="t200" suffix="rear_starboard_vertical"
+        xyz="-0.12 -0.22 0.06" rpy="0 ${radians(-90)} 0" turning_direction="ccw"
+        propeller_direction="ccw" color="grey" number="6" />
+    <xacro:thruster parent="base_link" model="t200" suffix="rear_port_vertical"
+        xyz="-0.12 0.22 0.06" rpy="0 ${radians(-90)} 0" turning_direction="cw"
+        propeller_direction="ccw" color="grey" number="7" />
+    <xacro:if value="$(arg use_vertical_camera)">
+        <xacro:camera_macro parent="base_link"
+            prefix="vertical_camera" xyz="${vertical_camera_position}"
+            rpy="${vertical_camera_orientation}" />
+    </xacro:if>
+    <xacro:if value="$(arg use_front_camera)">
+        <xacro:camera_macro parent="base_link"
+            prefix="front_camera" xyz="${front_camera_position}"
+            rpy="${front_camera_orientation}" />
+    </xacro:if>
     <gazebo>
         <plugin filename="buoyancy" name="hippo_gz_plugins::buoyancy">

Commit message: make the simulation behave more nicely

File: models/bluerov/urdf/bluerov.xacro (robot description, xacro)
@@ -61,7 +61,7 @@
             <buoyancy>
                 <link_name>base_link</link_name>
-                <origin>0 0 0.01</origin>
+                <origin>${buoyancy_origin}</origin>
                 <force_added>0</force_added>
-                <compensation>1.01</compensation>
+                <compensation>${buoyancy_compensation}</compensation>
                 <height_scale_limit>0.1</height_scale_limit>
             </buoyancy>

File: models/thruster/urdf/t200_params.xacro (robot description, xacro)
@@ -7,5 +7,5 @@
     <!-- based on 14V performance data and forced interception at 0.0 -->
     <xacro:property name="thrust_quadratic_coeff" value="0.015547" />
-    <xacro:property name="thrust_linear_coeff" value="-0.04243" />
+    <xacro:property name="thrust_linear_coeff" value="0.04243" />
     <xacro:property name="thrust_constant_coeff" value="0.0" />
     <xacro:property name="torque_constant" value="0.0" />
