Commit message: commit before rebase, changed added buoyancy for manipulator compensation

File: models/bluerov/urdf/bluerov_params_uvms.xacro (robot description, xacro)
@@ -10,6 +10,12 @@
     <xacro:property name="damping_angular" value="0.3 0.3 0.3" />
     <!-- alpha manipulator weight underwater: 1.272 kg - 0.5719 kg = 0.7001  => 0.7001 / 11.0 (mass bluerov) = 0.064-->
-    <xacro:property name="buoyancy_compensation" value="1.065" /> <!--1.001 default -->
-    <xacro:property name="buoyancy_origin" value="0 0 0.05" />
+    <xacro:property name="buoyancy_compensation_AUV" value="1.001" /> <!--1.001 default -->
+    <xacro:property name="buoyancy_origin_AUV" value="${[0, 0, 0.005]}" />
+    <xacro:property name="buoyancy_compensation_added" value="0.064" /> <!-- must be the same as for controller! -->
+    <xacro:property name="buoyancy_origin_added" value="${[0, 0, 0.05]}" />
+    <xacro:property name="buoyancy_compensation" value="${buoyancy_compensation_AUV + buoyancy_compensation_added}" /> <!--1.001 default -->
+    <xacro:property name="buoyancy_origin" value="${buoyancy_origin_AUV[0] * buoyancy_compensation_AUV + buoyancy_origin_added[0] * buoyancy_compensation_added / (buoyancy_compensation_AUV + buoyancy_compensation_added)}
+            ${buoyancy_origin_AUV[1] * buoyancy_compensation_AUV + buoyancy_origin_added[1] * buoyancy_compensation_added / (buoyancy_compensation_AUV + buoyancy_compensation_added)}
+            ${buoyancy_origin_AUV[2] * buoyancy_compensation_AUV + buoyancy_origin_added[2] * buoyancy_compensation_added / (buoyancy_compensation_AUV + buoyancy_compensation_added)}" />
     <xacro:property name="barometer_position" value="-0.15 0 -0.05" />
     <xacro:property name="barometer_noise" value="100.0" />
@@ -18,13 +24,4 @@
     <xacro:property name="imu_orientation" value="${radians(0)} ${radians(0)} ${radians(0)}"/>
     <xacro:property name="imu_noise" value="0.0003"/>
-    <xacro:property name="range_sensor_position" value="0.2 0 0.1" />
-    <xacro:property name="range_sensor_orientation" value="${radians(0)} ${radians(0)} ${radians(0)}" />
-    <xacro:arg name="use_vertical_camera" default="false" />
-    <xacro:property name="vertical_camera_position" value="0.15 0 -0.08" />
-    <xacro:property name="vertical_camera_orientation" value="0 ${radians(90)} 0" />
-    <xacro:arg name="use_front_camera" default="false" />
-    <!-- probably we want this to be the same as the range sensor position -->
-    <xacro:property name="front_camera_position" value="0.2 0 0.1" />
-    <xacro:property name="front_camera_orientation" value="0 0 0" />
     <xacro:property name="thruster_r" value="0.097" />
 </robot>

Commit message: move bluerov xacro to macro

File: models/bluerov/urdf/bluerov_params_uvms.xacro (robot description, xacro)
@@ -9,6 +9,13 @@
     <xacro:property name="damping_linear" value="7 7 7" />
     <xacro:property name="damping_angular" value="0.3 0.3 0.3" />
-    <xacro:property name="buoyancy_compensation" value="1.001" />
-    <xacro:property name="buoyancy_origin" value="0 0 0.005" />
+    <!--  0.899 / 11.0 (mass bluerov) = 0.0817-->
+    <xacro:property name="buoyancy_compensation_AUV" value="1.001" /> <!--1.001 default -->
+    <xacro:property name="buoyancy_origin_AUV" value="${[0, 0, 0.005]}" />
+    <xacro:property name="buoyancy_compensation_added" value="0.0817" /> <!-- must be the same as for controller! -->
+    <xacro:property name="buoyancy_origin_added" value="${[0, 0, 0.05]}" />
+    <xacro:property name="buoyancy_compensation" value="${buoyancy_compensation_AUV + buoyancy_compensation_added}" />
+    <xacro:property name="buoyancy_origin" value="${(buoyancy_origin_AUV[0] * buoyancy_compensation_AUV + buoyancy_origin_added[0] * buoyancy_compensation_added) / (buoyancy_compensation_AUV + buoyancy_compensation_added)}
+            ${(buoyancy_origin_AUV[1] * buoyancy_compensation_AUV + buoyancy_origin_added[1] * buoyancy_compensation_added) / (buoyancy_compensation_AUV + buoyancy_compensation_added)}
+            ${(buoyancy_origin_AUV[2] * buoyancy_compensation_AUV + buoyancy_origin_added[2] * buoyancy_compensation_added) / (buoyancy_compensation_AUV + buoyancy_compensation_added)}" />
     <xacro:property name="barometer_position" value="-0.15 0 -0.05" />
     <xacro:property name="barometer_noise" value="100.0" />
@@ -17,4 +24,5 @@
     <xacro:property name="imu_orientation" value="${radians(0)} ${radians(0)} ${radians(0)}"/>
     <xacro:property name="imu_noise" value="0.0003"/>
+    <xacro:property name="thruster_r" value="0.097" />
     <xacro:arg name="use_range_sensor" default="false" />
     <xacro:property name="range_sensor_position" value="0.2 0 0.1" />

File: models/bluerov/urdf/bluerov_rviz.xacro (robot description, xacro)
@@ -2,6 +2,5 @@
 <robot xmlns:xacro="http://www.ros.org/wiki/xacro" name="hippocampus">
     <xacro:arg name="base_link_name" default="base_link"/>
-    <xacro:arg name="vehicle_name" default="bluerov"/>
     <xacro:include filename="$(find hippo_sim)/models/bluerov/urdf/bluerov_macro.xacro"/>
-    <xacro:bluerov base_link_name="$(arg base_link_name)" link_ns="$(arg vehicle_name)" />
+    <xacro:bluerov base_link_name="$(arg base_link_name)" link_ns="$(arg vehicle_name)" rviz_model="True"/>
 </robot>

File: models/camera/urdf/camera_macro.xacro (robot description, xacro)
@@ -4,6 +4,6 @@
         <xacro:include filename="$(find hippo_sim)/models/common/urdf/common.xacro" />
         <xacro:include filename="$(find hippo_sim)/models/camera/urdf/camera_params.xacro" />
-        <xacro:property name="link" value="${prefix}_link" />
-        <xacro:property name="joint" value="${prefix}_joint" />
+        <xacro:property name="link" value="$(arg vehicle_name)/${prefix}_link" />
+        <xacro:property name="joint" value="$(arg vehicle_name)/${prefix}_joint" />
         <link name="${link}">
             <xacro:zero_inertia />
@@ -32,5 +32,5 @@
                 </material>
             </visual>
-            <sensor name="${prefix}" type="camera">
+            <sensor name="$(arg vehicle_name)_${prefix}" type="camera">
                 <camera>
                     <camera_info_topic>$(arg vehicle_name)/${prefix}/camera_info</camera_info_topic>
