Commit message: added files for bluerov control, viz and bringup, bridge clock topic

File: models/bluerov/urdf/bluerov_macro.xacro (robot description, xacro)
@@ -1,6 +1,11 @@
 <?xml version="1.0"?>
 <robot xmlns:xacro="http://www.ros.org/wiki/xacro" name="hippocampus">
-    <xacro:macro name="bluerov" params="base_link_name:=base_link">
-        <xacro:include filename="$(find hippo_sim)/models/bluerov/urdf/bluerov_params.xacro" />
+    <xacro:macro name="bluerov" params="base_link_name:=base_link use_uvms_param:=False">
+        <xacro:if value="${use_uvms_param == True}">
+            <xacro:include filename="$(find hippo_sim)/models/bluerov/urdf/bluerov_params_uvms.xacro" />
+        </xacro:if>
+        <xacro:unless value="${use_uvms_param == True}">
+            <xacro:include filename="$(find hippo_sim)/models/bluerov/urdf/bluerov_params.xacro" />
+        </xacro:unless>
         <xacro:include filename="$(find hippo_sim)/models/thruster/urdf/thruster_macro.xacro" />
         <xacro:include filename="$(find hippo_sim)/models/hippo3/urdf/mount_macro.xacro" />

File: models/bluerov/urdf/bluerov_params_uvms.xacro (robot description, xacro)
@@ -9,6 +9,7 @@
     <xacro:property name="damping_linear" value="7 7 7" />
     <xacro:property name="damping_angular" value="0.3 0.3 0.3" />
-    <xacro:property name="buoyancy_compensation" value="1.001" />
-    <xacro:property name="buoyancy_origin" value="0 0 -0.1" />
+    <!-- alpha manipulator weight underwater: 1.272 kg - 0.5719 kg = 0.7001  => 0.7001 / 11.0 (mass bluerov) = 0.064-->
+    <xacro:property name="buoyancy_compensation" value="1.065" /> <!--1.001 default -->
+    <xacro:property name="buoyancy_origin" value="0 0 0.05" />
     <xacro:property name="barometer_position" value="-0.15 0 -0.05" />
     <xacro:property name="barometer_noise" value="100.0" />

Commit message: bug fix in buoyancy torque calculatieon, rviz integration for xacro files, map_body broadcaster

File: models/bluerov/urdf/bluerov_macro.xacro (robot description, xacro)
@@ -1,5 +1,5 @@
 <?xml version="1.0"?>
 <robot xmlns:xacro="http://www.ros.org/wiki/xacro" name="hippocampus">
-    <xacro:macro name="bluerov" params="base_link_name:=base_link use_uvms_param:=False">
+    <xacro:macro name="bluerov" params="base_link_name:=base_link use_uvms_param:=False rviz_model:=False">
         <xacro:if value="${use_uvms_param == True}">
             <xacro:include filename="$(find hippo_sim)/models/bluerov/urdf/bluerov_params_uvms.xacro" />
@@ -17,22 +17,26 @@
         </gazebo>
         <link name="${base_link_name}">
+            <xacro:unless value="${rviz_model == True}">
             <inertial name="base_link_inertial">
                 <mass value="${base_mass}" />
                 <inertia ixx="${ixx}" ixy="0.0" ixz="0.0" iyy="${iyy}" iyz="0.0" izz="${izz}" />
             </inertial>
+            </xacro:unless>
             <visual name="base_link_visual">
                 <geometry>
-                    <mesh filename="$(find hippo_sim)/models/bluerov/meshes/bluerov.dae" />
+                    <mesh filename="file://$(find hippo_sim)/models/bluerov/meshes/bluerov.dae" />
                 </geometry>
             </visual>
         </link>
-        <xacro:thruster parent="${base_link_name}" model="t200" suffix="front_starboard_horizontal" xyz="0.14 -0.10 0" rpy="0 0 ${radians(45)}" turning_direction="cw" propeller_direction="ccw" color="red" number="0" />
-        <xacro:thruster parent="${base_link_name}" model="t200" suffix="front_port_horizontal" xyz="0.14 0.10 0" rpy="0 0 ${radians(-45)}" turning_direction="cw" propeller_direction="ccw" color="green" number="1" />
-        <xacro:thruster parent="${base_link_name}" model="t200" suffix="rear_starboard_horizontal" xyz="-0.14 -0.10 0" rpy="0 0 ${radians(135)}" turning_direction="cw" propeller_direction="cw" color="grey" number="2" />
-        <xacro:thruster parent="${base_link_name}" model="t200" suffix="rear_port_horizontal" xyz="-0.14 0.10 0" rpy="0 0 ${radians(-135)}" turning_direction="cw" propeller_direction="cw" color="grey" number="3" />
-        <xacro:thruster parent="${base_link_name}" model="t200" suffix="front_starboard_vertical" xyz="0.12 -0.22 0.06" rpy="0 ${radians(-90)} 0" turning_direction="cw" propeller_direction="ccw" color="red" number="4" />
-        <xacro:thruster parent="${base_link_name}" model="t200" suffix="front_port_vertical" xyz="0.12 0.22 0.06" rpy="0 ${radians(-90)} 0" turning_direction="ccw" propeller_direction="ccw" color="green" number="5" />
-        <xacro:thruster parent="${base_link_name}" model="t200" suffix="rear_starboard_vertical" xyz="-0.12 -0.22 0.06" rpy="0 ${radians(-90)} 0" turning_direction="ccw" propeller_direction="ccw" color="grey" number="6" />
-        <xacro:thruster parent="${base_link_name}" model="t200" suffix="rear_port_vertical" xyz="-0.12 0.22 0.06" rpy="0 ${radians(-90)} 0" turning_direction="cw" propeller_direction="ccw" color="grey" number="7" />
+        <xacro:unless value="${rviz_model == True}">
+            <xacro:thruster parent="${base_link_name}" model="t200" suffix="front_starboard_horizontal" xyz="0.14 -0.10 0" rpy="0 0 ${radians(45)}" turning_direction="cw" propeller_direction="ccw" color="red" number="0"/>
+            <xacro:thruster parent="${base_link_name}" model="t200" suffix="front_port_horizontal" xyz="0.14 0.10 0" rpy="0 0 ${radians(-45)}" turning_direction="cw" propeller_direction="ccw" color="green" number="1" />
+            <xacro:thruster parent="${base_link_name}" model="t200" suffix="rear_starboard_horizontal" xyz="-0.14 -0.10 0" rpy="0 0 ${radians(135)}" turning_direction="cw" propeller_direction="cw" color="grey" number="2" />
+            <xacro:thruster parent="${base_link_name}" model="t200" suffix="rear_port_horizontal" xyz="-0.14 0.10 0" rpy="0 0 ${radians(-135)}" turning_direction="cw" propeller_direction="cw" color="grey" number="3" />
+            <xacro:thruster parent="${base_link_name}" model="t200" suffix="front_starboard_vertical" xyz="0.12 -0.22 0.06" rpy="0 ${radians(-90)} 0" turning_direction="cw" propeller_direction="ccw" color="red" number="4" />
+            <xacro:thruster parent="${base_link_name}" model="t200" suffix="front_port_vertical" xyz="0.12 0.22 0.06" rpy="0 ${radians(-90)} 0" turning_direction="ccw" propeller_direction="ccw" color="green" number="5" />
+            <xacro:thruster parent="${base_link_name}" model="t200" suffix="rear_starboard_vertical" xyz="-0.12 -0.22 0.06" rpy="0 ${radians(-90)} 0" turning_direction="ccw" propeller_direction="ccw" color="grey" number="6" />
+            <xacro:thruster parent="${base_link_name}" model="t200" suffix="rear_port_vertical" xyz="-0.12 0.22 0.06" rpy="0 ${radians(-90)} 0" turning_direction="cw" propeller_direction="ccw" color="grey" number="7" />
+        </xacro:unless>
         <gazebo>
             <plugin filename="buoyancy" name="hippo_gz_plugins::buoyancy">

File: models/bluerov/urdf/bluerov_params.xacro (robot description, xacro)
@@ -10,5 +10,5 @@
     <xacro:property name="damping_angular" value="0.3 0.3 0.3" />
     <xacro:property name="buoyancy_compensation" value="1.001" />
-    <xacro:property name="buoyancy_origin" value="0 0 -0.1" />
+    <xacro:property name="buoyancy_origin" value="0 0 0.005" />
     <xacro:property name="barometer_position" value="-0.15 0 -0.05" />
     <xacro:property name="barometer_noise" value="100.0" />

Commit message: added bluerov velocity controller, preparation for uvms integration

File: models/bluerov/urdf/bluerov_macro.xacro (robot description, xacro)
@@ -42,5 +42,5 @@
             <plugin filename="buoyancy" name="hippo_gz_plugins::buoyancy">
                 <buoyancy>
-                    <link_name>base_link</link_name>
+                    <link_name>${base_link_name}</link_name>
                     <origin>${buoyancy_origin}</origin>
                     <force_added>0</force_added>
@@ -51,5 +51,5 @@
             <plugin filename="hydrodynamics" name="hippo_gz_plugins::hydrodynamics">
                 <hydrodynamics>
-                    <link>base_link</link>
+                    <link>${base_link_name}</link>
                     <added_mass_linear>${added_mass_linear}</added_mass_linear>
                     <added_mass_angular>${added_mass_angular}</added_mass_angular>
@@ -59,10 +59,10 @@
             </plugin>
             <plugin filename="pose" name="hippo_gz_plugins::pose">
-                <link>base_link</link>
+                <link>${base_link_name}</link>
                 <update_rate>50.0</update_rate>
                 <base_topic>ground_truth/pose</base_topic>
             </plugin>
             <plugin filename="odometry" name="hippo_gz_plugins::odometry">
-                <link>base_link</link>
+                <link>${base_link_name}</link>
                 <update_rate>50.0</update_rate>
                 <base_topic>ground_truth/odometry</base_topic>
@@ -70,5 +70,5 @@
             <!--
             <plugin filename="barometer" name="hippo_gz_plugins::barometer">
-                <link>base_link</link>
+                <link>${base_link_name}</link>
                 <update_rate>100.0</update_rate>
                 <base_topic>pressure</base_topic>
@@ -78,21 +78,21 @@
             </plugin>
             <plugin filename="range_sensor" name="hippo_gz_plugins::range_sensor">
-                <link>base_link</link>
+                <link>${base_link_name}</link>
                 <range_topic>range_topic</range_topic>
                 <update_rate>20.0</update_rate>
                 <model name="range_tag_00">
-                    <link>base_link</link>
+                    <link>${base_link_name}</link>
                     <id>0</id>
                 </model>
                 <model name="range_tag_01">
-                    <link>base_link</link>
+                    <link>${base_link_name}</link>
                     <id>1</id>
                 </model>
                 <model name="range_tag_02">
-                    <link>base_link</link>
+                    <link>${base_link_name}</link>
                     <id>2</id>
                 </model>
                 <model name="range_tag_03">
-                    <link>base_link</link>
+                    <link>${base_link_name}</link>
                     <id>3</id>
                 </model>

Commit message: kinematic control pipeline works, gazebo not accurate in setting link velocities

File: models/bluerov/urdf/bluerov_macro.xacro (robot description, xacro)
@@ -1,5 +1,5 @@
 <?xml version="1.0"?>
 <robot xmlns:xacro="http://www.ros.org/wiki/xacro" name="hippocampus">
-    <xacro:macro name="bluerov" params="base_link_name:=base_link use_uvms_param:=False rviz_model:=False">
+    <xacro:macro name="bluerov" params="base_link_name:=base_link use_uvms_param:=False rviz_model:=False simulate_kinematics:=False">
         <xacro:if value="${use_uvms_param == True}">
             <xacro:include filename="$(find hippo_sim)/models/bluerov/urdf/bluerov_params_uvms.xacro" />
@@ -40,22 +40,29 @@
         </xacro:unless>
         <gazebo>
-            <plugin filename="buoyancy" name="hippo_gz_plugins::buoyancy">
-                <buoyancy>
+            <xacro:if value="${simulate_kinematics == True}">
+                <plugin filename="kinematic_control" name="hippo_gz_plugins::kinematic_control">
                     <link_name>${base_link_name}</link_name>
-                    <origin>${buoyancy_origin}</origin>
-                    <force_added>0</force_added>
-                    <compensation>${buoyancy_compensation}</compensation> <!-- 1.01 -->
-                    <height_scale_limit>0.1</height_scale_limit>
-                </buoyancy>
-            </plugin>
-            <plugin filename="hydrodynamics" name="hippo_gz_plugins::hydrodynamics">
-                <hydrodynamics>
-                    <link>${base_link_name}</link>
-                    <added_mass_linear>${added_mass_linear}</added_mass_linear>
-                    <added_mass_angular>${added_mass_angular}</added_mass_angular>
-                    <damping_linear>${damping_linear}</damping_linear>
-                    <damping_angular>${damping_angular}</damping_angular>
-                </hydrodynamics>
-            </plugin>
+                </plugin>
+            </xacro:if>
+            <xacro:unless value="${simulate_kinematics == True}">
+                <plugin filename="buoyancy" name="hippo_gz_plugins::buoyancy">
+                    <buoyancy>
+                        <link_name>${base_link_name}</link_name>
+                        <origin>${buoyancy_origin}</origin>
+                        <force_added>0</force_added>
+                        <compensation>${buoyancy_compensation}</compensation> <!-- 1.01 -->
+                        <height_scale_limit>0.1</height_scale_limit>
+                    </buoyancy>
+                </plugin>
+                <plugin filename="hydrodynamics" name="hippo_gz_plugins::hydrodynamics">
+                    <hydrodynamics>
+                        <link>${base_link_name}</link>
+                        <added_mass_linear>${added_mass_linear}</added_mass_linear>
+                        <added_mass_angular>${added_mass_angular}</added_mass_angular>
+                        <damping_linear>${damping_linear}</damping_linear>
+                        <damping_angular>${damping_angular}</damping_angular>
+                    </hydrodynamics>
+                </plugin>
+            </xacro:unless>
             <plugin filename="pose" name="hippo_gz_plugins::pose">
                 <link>${base_link_name}</link>

Commit message: added physical mapping for BlueROV thruster

File: models/bluerov/urdf/bluerov_macro.xacro (robot description, xacro)
@@ -30,4 +30,5 @@
         </link>
         <xacro:unless value="${rviz_model == True}">
+            <!--
             <xacro:thruster parent="${link_ns}${base_link_name}" model="t200" suffix="front_starboard_horizontal" xyz="0.14 -0.10 0" rpy="0 0 ${radians(45)}" turning_direction="cw" propeller_direction="ccw" color="red" number="0"/>
             <xacro:thruster parent="${link_ns}${base_link_name}" model="t200" suffix="front_port_horizontal" xyz="0.14 0.10 0" rpy="0 0 ${radians(-45)}" turning_direction="cw" propeller_direction="ccw" color="green" number="1" />
@@ -38,4 +39,13 @@
             <xacro:thruster parent="${link_ns}${base_link_name}" model="t200" suffix="rear_starboard_vertical" xyz="-0.12 -0.22 0.06" rpy="0 ${radians(-90)} 0" turning_direction="ccw" propeller_direction="ccw" color="grey" number="6" />
             <xacro:thruster parent="${link_ns}${base_link_name}" model="t200" suffix="rear_port_vertical" xyz="-0.12 0.22 0.06" rpy="0 ${radians(-90)} 0" turning_direction="cw" propeller_direction="ccw" color="grey" number="7" />
+            -->
+            <xacro:thruster parent="${link_ns}${base_link_name}" model="t200" suffix="front_starboard_horizontal" xyz="0.132 -0.10 0" rpy="0 0 ${radians(42)}" turning_direction="cw" propeller_direction="ccw" color="red" number="0"/>
+            <xacro:thruster parent="${link_ns}${base_link_name}" model="t200" suffix="front_port_horizontal" xyz="0.132 -0.10 0" rpy="0 0 ${radians(-42)}" turning_direction="cw" propeller_direction="ccw" color="green" number="1" />
+            <xacro:thruster parent="${link_ns}${base_link_name}" model="t200" suffix="rear_starboard_horizontal" xyz="-0.149 -0.0998 0" rpy="0 0 ${radians(133)}" turning_direction="cw" propeller_direction="cw" color="grey" number="2" />
+            <xacro:thruster parent="${link_ns}${base_link_name}" model="t200" suffix="rear_port_horizontal" xyz="-0.149 0.0998 0" rpy="0 0 ${radians(-133)}" turning_direction="cw" propeller_direction="cw" color="grey" number="3" />
+            <xacro:thruster parent="${link_ns}${base_link_name}" model="t200" suffix="front_starboard_vertical" xyz="0.12 -0.218 0.06" rpy="0 ${radians(-90)} 0" turning_direction="cw" propeller_direction="ccw" color="red" number="4" />
+            <xacro:thruster parent="${link_ns}${base_link_name}" model="t200" suffix="front_port_vertical" xyz="0.12 0.218 0.06" rpy="0 ${radians(-90)} 0" turning_direction="ccw" propeller_direction="ccw" color="green" number="5" />
+            <xacro:thruster parent="${link_ns}${base_link_name}" model="t200" suffix="rear_starboard_vertical" xyz="-0.12 -0.218 0.06" rpy="0 ${radians(-90)} 0" turning_direction="ccw" propeller_direction="ccw" color="grey" number="6" />
+            <xacro:thruster parent="${link_ns}${base_link_name}" model="t200" suffix="rear_port_vertical" xyz="-0.12 0.218 0.06" rpy="0 ${radians(-90)} 0" turning_direction="cw" propeller_direction="ccw" color="grey" number="7" />
         </xacro:unless>
         <gazebo>

File: models/bluerov/urdf/bluerov_params_uvms.xacro (robot description, xacro)
@@ -9,13 +9,17 @@
     <xacro:property name="damping_linear" value="7 7 7" />
     <xacro:property name="damping_angular" value="0.3 0.3 0.3" />
-    <!-- alpha manipulator weight underwater: 1.272 kg - 0.5719 kg = 0.7001  => 0.7001 / 11.0 (mass bluerov) = 0.064-->
+    <!-- alpha manipulator weight underwater: 1.405 kg - 0.6206 kg = 0.7001  => 0.7844 / 11.0 (mass bluerov) = 0.0713-->
     <xacro:property name="buoyancy_compensation_AUV" value="1.001" /> <!--1.001 default -->
     <xacro:property name="buoyancy_origin_AUV" value="${[0, 0, 0.005]}" />
-    <xacro:property name="buoyancy_compensation_added" value="0.064" /> <!-- must be the same as for controller! -->
+    <xacro:property name="buoyancy_compensation_added" value="0.0713" /> <!-- must be the same as for controller! -->
     <xacro:property name="buoyancy_origin_added" value="${[0, 0, 0.05]}" />
-    <xacro:property name="buoyancy_compensation" value="${buoyancy_compensation_AUV + buoyancy_compensation_added}" /> <!--1.001 default -->
-    <xacro:property name="buoyancy_origin" value="${buoyancy_origin_AUV[0] * buoyancy_compensation_AUV + buoyancy_origin_added[0] * buoyancy_compensation_added / (buoyancy_compensation_AUV + buoyancy_compensation_added)}
-            ${buoyancy_origin_AUV[1] * buoyancy_compensation_AUV + buoyancy_origin_added[1] * buoyancy_compensation_added / (buoyancy_compensation_AUV + buoyancy_compensation_added)}
-            ${buoyancy_origin_AUV[2] * buoyancy_compensation_AUV + buoyancy_origin_added[2] * buoyancy_compensation_added / (buoyancy_compensation_AUV + buoyancy_compensation_added)}" />
+    <!--
+    <xacro:property name="buoyancy_compensation" value="${buoyancy_compensation_AUV + buoyancy_compensation_added}" />
+    <xacro:property name="buoyancy_origin" value="${(buoyancy_origin_AUV[0] * buoyancy_compensation_AUV + buoyancy_origin_added[0] * buoyancy_compensation_added) / (buoyancy_compensation_AUV + buoyancy_compensation_added)}
+            ${(buoyancy_origin_AUV[1] * buoyancy_compensation_AUV + buoyancy_origin_added[1] * buoyancy_compensation_added) / (buoyancy_compensation_AUV + buoyancy_compensation_added)}
+            ${(buoyancy_origin_AUV[2] * buoyancy_compensation_AUV + buoyancy_origin_added[2] * buoyancy_compensation_added) / (buoyancy_compensation_AUV + buoyancy_compensation_added)}" />
+    -->
+    <xacro:property name="buoyancy_compensation" value="${buoyancy_compensation_AUV}"/>
+    <xacro:property name="buoyancy_origin" value="${buoyancy_origin_AUV[0]} ${buoyancy_origin_AUV[1]} ${buoyancy_origin_AUV[2]}"/>
     <xacro:property name="barometer_position" value="-0.15 0 -0.05" />
     <xacro:property name="barometer_noise" value="100.0" />

File: models/thruster/urdf/t200_params.xacro (robot description, xacro)
@@ -12,6 +12,6 @@
     <!-- for reversed direction:  0.01268 -0.05067 0.0 -->
     <!-- Throttle = f(revs/s) -->
-    <xacro:property name="velocity_quadratic_coeff" value="1.2679e-4"/>
-    <xacro:property name="velocity_linear_coeff" value="1.1105e-2"/>
+    <xacro:property name="velocity_quadratic_coeff" value="0.00914"/>
+    <xacro:property name="velocity_linear_coeff" value="-0.2228"/>
     <xacro:property name="velocity_constant_coeff" value="0.0"/>
     <xacro:property name="rpm_scaler" value="10" />
