Commit message: commit before upstream pull request

File: models/bluerov/urdf/bluerov_macro.xacro (robot description, xacro)
@@ -30,14 +30,4 @@
         </link>
         <xacro:unless value="${rviz_model == True}">
-            <!--
-            <xacro:thruster parent="${link_ns}${base_link_name}" model="t200" suffix="front_starboard_horizontal" xyz="0.14 -0.10 0" rpy="0 0 ${radians(45)}" turning_direction="cw" propeller_direction="ccw" color="red" number="0"/>
-            <xacro:thruster parent="${link_ns}${base_link_name}" model="t200" suffix="front_port_horizontal" xyz="0.14 0.10 0" rpy="0 0 ${radians(-45)}" turning_direction="cw" propeller_direction="ccw" color="green" number="1" />
-            <xacro:thruster parent="${link_ns}${base_link_name}" model="t200" suffix="rear_starboard_horizontal" xyz="-0.14 -0.10 0" rpy="0 0 ${radians(135)}" turning_direction="cw" propeller_direction="cw" color="grey" number="2" />
-            <xacro:thruster parent="${link_ns}${base_link_name}" model="t200" suffix="rear_port_horizontal" xyz="-0.14 0.10 0" rpy="0 0 ${radians(-135)}" turning_direction="cw" propeller_direction="cw" color="grey" number="3" />
-            <xacro:thruster parent="${link_ns}${base_link_name}" model="t200" suffix="front_starboard_vertical" xyz="0.12 -0.22 0.06" rpy="0 ${radians(-90)} 0" turning_direction="cw" propeller_direction="ccw" color="red" number="4" />
-            <xacro:thruster parent="${link_ns}${base_link_name}" model="t200" suffix="front_port_vertical" xyz="0.12 0.22 0.06" rpy="0 ${radians(-90)} 0" turning_direction="ccw" propeller_direction="ccw" color="green" number="5" />
-            <xacro:thruster parent="${link_ns}${base_link_name}" model="t200" suffix="rear_starboard_vertical" xyz="-0.12 -0.22 0.06" rpy="0 ${radians(-90)} 0" turning_direction="ccw" propeller_direction="ccw" color="grey" number="6" />
-            <xacro:thruster parent="${link_ns}${base_link_name}" model="t200" suffix="rear_port_vertical" xyz="-0.12 0.22 0.06" rpy="0 ${radians(-90)} 0" turning_direction="cw" propeller_direction="ccw" color="grey" number="7" />
-            -->
             <xacro:thruster parent="${link_ns}${base_link_name}" model="t200" suffix="front_starboard_horizontal" xyz="0.132 -0.10 0" rpy="0 0 ${radians(42)}" turning_direction="cw" propeller_direction="ccw" color="red" number="0"/>
             <xacro:thruster parent="${link_ns}${base_link_name}" model="t200" suffix="front_port_horizontal" xyz="0.132 -0.10 0" rpy="0 0 ${radians(-42)}" turning_direction="cw" propeller_direction="ccw" color="green" number="1" />

File: models/bluerov/urdf/bluerov_params_uvms.xacro (robot description, xacro)
@@ -18,8 +18,4 @@
             ${(buoyancy_origin_AUV[1] * buoyancy_compensation_AUV + buoyancy_origin_added[1] * buoyancy_compensation_added) / (buoyancy_compensation_AUV + buoyancy_compensation_added)}
             ${(buoyancy_origin_AUV[2] * buoyancy_compensation_AUV + buoyancy_origin_added[2] * buoyancy_compensation_added) / (buoyancy_compensation_AUV + buoyancy_compensation_added)}" />
-    <!--
-    <xacro:property name="buoyancy_compensation" value="${buoyancy_compensation_AUV}"/>
-    <xacro:property name="buoyancy_origin" value="${buoyancy_origin_AUV[0]} ${buoyancy_origin_AUV[1]} ${buoyancy_origin_AUV[2]}"/>
-    -->
     <xacro:property name="barometer_position" value="-0.15 0 -0.05" />
     <xacro:property name="barometer_noise" value="100.0" />

Commit message: fixed non-adaptable base link name for range sensor

File: models/bluerov/urdf/bluerov_macro.xacro (robot description, xacro)
@@ -1,7 +1,9 @@
 <?xml version="1.0"?>
 <robot xmlns:xacro="http://www.ros.org/wiki/xacro" name="hippocampus">
-    <xacro:macro name="bluerov" params="base_link_name:=base_link link_ns use_uvms_param:=False rviz_model:=False simulate_kinematics:=False">
+    <xacro:macro name="bluerov"
+        params="base_link_name:=base_link link_ns use_uvms_param:=False rviz_model:=False simulate_kinematics:=False">
         <xacro:if value="${use_uvms_param == True}">
-            <xacro:include filename="$(find hippo_sim)/models/bluerov/urdf/bluerov_params_uvms.xacro" />
+            <xacro:include
+                filename="$(find hippo_sim)/models/bluerov/urdf/bluerov_params_uvms.xacro" />
         </xacro:if>
         <xacro:unless value="${use_uvms_param == True}">
@@ -9,5 +11,6 @@
         </xacro:unless>
         <xacro:include filename="$(find hippo_sim)/models/bluerov/urdf/bluerov_thrusters.xacro" />
-        <!-- <xacro:include filename="$(find hippo_sim)/models/range_sensor/urdf/range_sensor_macro.xacro" /> -->
+        <!-- <xacro:include filename="$(find
+        hippo_sim)/models/range_sensor/urdf/range_sensor_macro.xacro" /> -->
         <xacro:include filename="$(find hippo_sim)/models/camera/urdf/camera_macro.xacro" />
         <xacro:property name="thruster_xy" value="${thruster_r / 2**0.5}" />
@@ -17,8 +20,8 @@
         <link name="${link_ns}/${base_link_name}">
             <xacro:unless value="${rviz_model == True}">
-            <inertial name="base_link_inertial">
-                <mass value="${base_mass}" />
-                <inertia ixx="${ixx}" ixy="0.0" ixz="0.0" iyy="${iyy}" iyz="0.0" izz="${izz}" />
-            </inertial>
+                <inertial name="base_link_inertial">
+                    <mass value="${base_mass}" />
+                    <inertia ixx="${ixx}" ixy="0.0" ixz="0.0" iyy="${iyy}" iyz="0.0" izz="${izz}" />
+                </inertial>
             </xacro:unless>
             <visual name="base_link_visual">
@@ -29,5 +32,5 @@
         </link>
         <xacro:unless value="${rviz_model == True}">
-            <xacro:bluerov_thrusters parent_link="${link_ns}/${base_link_name}"/>
+            <xacro:bluerov_thrusters parent_link="${link_ns}/${base_link_name}" />
             <xacro:if value="$(arg use_vertical_camera)">
                 <xacro:camera_macro parent="base_link"
@@ -47,5 +50,6 @@
                 </plugin>
                 <!--
-                <plugin name="ignition::gazebo::systems::VelocityControl" filename="ignition-gazebo-velocity-control-system">
+                <plugin name="ignition::gazebo::systems::VelocityControl"
+                filename="ignition-gazebo-velocity-control-system">
                     <link_name>${link_ns}/${base_link_name}</link_name>
                 </plugin>
@@ -92,5 +96,5 @@
             <xacro:if value="$(arg use_range_sensor)">
                 <plugin filename="range_sensor" name="hippo_gz_plugins::range_sensor">
-                    <link>base_link</link>
+                    <link>${link_ns}/${base_link_name}</link>
                     <range_topic>range_topic</range_topic>
                     <update_rate>10.0</update_rate>

Commit message: add acoustic modem link to bluerov and hippocampus model

File: models/bluerov/urdf/bluerov_macro.xacro (robot description, xacro)
@@ -14,4 +14,5 @@
         hippo_sim)/models/range_sensor/urdf/range_sensor_macro.xacro" /> -->
         <xacro:include filename="$(find hippo_sim)/models/camera/urdf/camera_macro.xacro" />
+        <xacro:include filename="$(find hippo_sim)/models/acoustic_modem/urdf/acoustic_modem_macro.xacro" />
         <xacro:property name="thruster_xy" value="${thruster_r / 2**0.5}" />
         <gazebo>
@@ -42,4 +43,9 @@
                     prefix="front_camera" xyz="${front_camera_position}"
                     rpy="${front_camera_orientation}" />
+            </xacro:if>
+            <xacro:if value="$(arg use_acoustic_modem)">
+                <xacro:acoustic_modem_macro parent="${link_ns}/${base_link_name}"
+                    prefix="${link_ns}/modem" xyz="${modem_position}"
+                    rpy="${modem_orientation}" />
             </xacro:if>
         </xacro:unless>

File: models/bluerov/urdf/bluerov_params.xacro (robot description, xacro)
@@ -27,4 +27,7 @@
     <xacro:property name="front_camera_position" value="0.2 0 0.1" />
     <xacro:property name="front_camera_orientation" value="0 0 0" />
+    <xacro:arg name="use_acoustic_modem" default="false"/>
+    <xacro:property name="modem_position" value="0 0 -0.3" />
+    <xacro:property name="modem_orientation" value="0 0 0" />
     <xacro:property name="thruster_r" value="0.097" />
 </robot>

File: models/bluerov/urdf/bluerov_params_uvms.xacro (robot description, xacro)
@@ -36,3 +36,6 @@
     <xacro:property name="front_camera_orientation" value="0 0 0" />
     <xacro:property name="thruster_r" value="0.097" />
+    <xacro:arg name="use_acoustic_modem" default="false" />
+    <xacro:property name="modem_position" value="0 0 -0.3" />
+    <xacro:property name="modem_orientation" value="0 0 0" />
 </robot>

File: models/hippo3/urdf/hippo3.xacro (robot description, xacro)
@@ -7,4 +7,5 @@
     <xacro:include filename="$(find hippo_sim)/models/hippo3/urdf/mount_macro.xacro" />
     <xacro:include filename="$(find hippo_sim)/models/camera/urdf/camera_macro.xacro" />
+    <xacro:include filename="$(find hippo_sim)/models/acoustic_modem/urdf/acoustic_modem_macro.xacro" />
     <xacro:property name="thruster_xy" value="${thruster_r / 2**0.5}" />
     <gazebo>
@@ -108,5 +109,10 @@
     <xacro:mount parent="base_link" suffix="starboard_bot" xyz="0 -${thruster_r / 2**0.5} -${thruster_r / 2**0.5}" rpy="${radians(135)} 0 0" />
     <xacro:mount parent="base_link" suffix="port_bot" xyz="0 ${thruster_r / 2**0.5} -${thruster_r / 2**0.5}" rpy="${radians(-135)} 0 0" />
-    <xacro:camera_macro parent="base_link" prefix="vertical_camera" xyz="${camera_position}" rpy="0 ${radians(90)} 0" />
+    <!-- <xacro:camera_macro parent="base_link" prefix="vertical_camera" xyz="${camera_position}" rpy="0 ${radians(90)} 0" /> -->
+    <xacro:if value="$(arg use_acoustic_modem)">
+        <xacro:acoustic_modem_macro parent="base_link"
+            prefix="modem" xyz="${modem_position}"
+            rpy="${modem_orientation}" />
+    </xacro:if>
     <gazebo>
         <plugin filename="buoyancy" name="hippo_gz_plugins::buoyancy">

File: models/hippo3/urdf/hippo3_params.xacro (robot description, xacro)
@@ -11,3 +11,6 @@
     <xacro:property name="damping_angular" value="0.00174 0.007 0.007"/>
     <xacro:property name="camera_position" value="0.15, 0.0 -0.03" />
+    <xacro:arg name="use_acoustic_modem" default="false" />
+    <xacro:property name="modem_position" value="0 0 -0.1" />
+    <xacro:property name="modem_orientation" value="0 0 0" />
 </robot>

Commit message: add use_vertical_camera param and actually use it for hippo, make camera_macro dumber

File: models/bluerov/urdf/bluerov_macro.xacro (robot description, xacro)
@@ -36,10 +36,14 @@
             <xacro:if value="$(arg use_vertical_camera)">
                 <xacro:camera_macro parent="${link_ns}/${base_link_name}"
-                    prefix="vertical_camera" xyz="${vertical_camera_position}"
+                    prefix="${link_ns}/vertical_camera" topic_prefix="${link_ns}/vertical_camera"
+                    ignition_frame_id="${link_ns}::vertical_camera"
+                    xyz="${vertical_camera_position}"
                     rpy="${vertical_camera_orientation}" />
             </xacro:if>
             <xacro:if value="$(arg use_front_camera)">
                 <xacro:camera_macro parent="${link_ns}/${base_link_name}"
-                    prefix="front_camera" xyz="${front_camera_position}"
+                    prefix="${link_ns}/front_camera" topic_prefix="${link_ns}/front_camera"
+                    ignition_frame_id="${link_ns}::front_camera"
+                    xyz="${front_camera_position}"
                     rpy="${front_camera_orientation}" />
             </xacro:if>

File: models/camera/urdf/camera_macro.xacro (robot description, xacro)
@@ -1,9 +1,9 @@
 <?xml version="1.0"?>
 <robot xmlns:xacro="http://www.ros.org/wiki/xacro">
-    <xacro:macro name="camera_macro" params="prefix parent xyz rpy">
+    <xacro:macro name="camera_macro" params="prefix parent topic_prefix ignition_frame_id xyz rpy">
         <xacro:include filename="$(find hippo_sim)/models/common/urdf/common.xacro" />
         <xacro:include filename="$(find hippo_sim)/models/camera/urdf/camera_params.xacro" />
-        <xacro:property name="link" value="$(arg vehicle_name)/${prefix}_link" />
-        <xacro:property name="joint" value="$(arg vehicle_name)/${prefix}_joint" />
+        <xacro:property name="link" value="${prefix}_link" />
+        <xacro:property name="joint" value="${prefix}_joint" />
         <link name="${link}">
             <xacro:zero_inertia />
@@ -32,5 +32,5 @@
                 </material>
             </visual>
-            <sensor name="$(arg vehicle_name)_${prefix}" type="camera">
+            <sensor name="${prefix}" type="camera">
                 <camera>
                     <noise>
@@ -39,5 +39,5 @@
                         <stddev>0.1</stddev>
                     </noise>
-                    <camera_info_topic>$(arg vehicle_name)/${prefix}/camera_info</camera_info_topic>
+                    <camera_info_topic>${prefix}/camera_info</camera_info_topic>
                     <horizontal_fov>${horizontal_fov}</horizontal_fov>
                     <image>
@@ -68,7 +68,7 @@
                 <update_rate>${fps}</update_rate>
                 <visualize>true</visualize>
-                <topic>$(arg vehicle_name)/${prefix}/image_rect</topic>
+                <topic>${topic_prefix}/image_rect</topic>
                 <!-- needs to be changed to gz_frame_id in the future -->
-                <ignition_frame_id>$(arg vehicle_name)::${prefix}</ignition_frame_id>
+                <ignition_frame_id>${ignition_frame_id}</ignition_frame_id>
             </sensor>
         </gazebo>

File: models/hippo3/urdf/hippo3.xacro (robot description, xacro)
@@ -109,5 +109,10 @@
     <xacro:mount parent="base_link" suffix="starboard_bot" xyz="0 -${thruster_r / 2**0.5} -${thruster_r / 2**0.5}" rpy="${radians(135)} 0 0" />
     <xacro:mount parent="base_link" suffix="port_bot" xyz="0 ${thruster_r / 2**0.5} -${thruster_r / 2**0.5}" rpy="${radians(-135)} 0 0" />
-    <!-- <xacro:camera_macro parent="base_link" prefix="vertical_camera" xyz="${camera_position}" rpy="0 ${radians(90)} 0" /> -->
+    <xacro:if value="$(arg use_vertical_camera)">
+        <xacro:camera_macro parent="base_link"
+            prefix="vertical_camera" topic_prefix="$(arg vehicle_name)/vertical_camera"
+            ignition_frame_id="$(arg vehicle_name)::vertical_camera"
+            xyz="${vertical_camera_position}" rpy="${vertical_camera_orientation}" />
+    </xacro:if>
     <xacro:if value="$(arg use_acoustic_modem)">
         <xacro:acoustic_modem_macro parent="base_link"

File: models/hippo3/urdf/hippo3_params.xacro (robot description, xacro)
@@ -10,5 +10,7 @@
     <xacro:property name="damping_linear" value="5.39 17.36 17.36"/>
     <xacro:property name="damping_angular" value="0.00174 0.007 0.007"/>
-    <xacro:property name="camera_position" value="0.15, 0.0 -0.03" />
+    <xacro:arg name="use_vertical_camera" default="false" />
+    <xacro:property name="vertical_camera_position" value="0.15, 0.0 -0.03" />
+    <xacro:property name="vertical_camera_orientation" value="0 ${radians(90)} 0" />
     <xacro:arg name="use_acoustic_modem" default="false" />
     <xacro:property name="modem_position" value="0 0 -0.1" />

Commit message: migration to jazzy/harmonic

File: models/bluerov/urdf/bluerov_macro.xacro (robot description, xacro)
@@ -60,5 +60,5 @@
                 </plugin>
                 <!--
-                <plugin name="ignition::gazebo::systems::VelocityControl"
+                <plugin name="gz::sim::systems::VelocityControl"
                 filename="ignition-gazebo-velocity-control-system">
                     <link_name>${link_ns}/${base_link_name}</link_name>

File: models/camera/urdf/camera_macro.xacro (robot description, xacro)
@@ -69,6 +69,5 @@
                 <visualize>true</visualize>
                 <topic>${topic_prefix}/image_rect</topic>
-                <!-- needs to be changed to gz_frame_id in the future -->
-                <ignition_frame_id>${ignition_frame_id}</ignition_frame_id>
+                <gz_frame_id>${ignition_frame_id}</gz_frame_id>
             </sensor>
         </gazebo>

File: models/hippo3/urdf/hippo3_params.xacro (robot description, xacro)
@@ -11,5 +11,5 @@
     <xacro:property name="damping_angular" value="0.00174 0.007 0.007"/>
     <xacro:arg name="use_vertical_camera" default="false" />
-    <xacro:property name="vertical_camera_position" value="0.15, 0.0 -0.03" />
+    <xacro:property name="vertical_camera_position" value="0.15 0.0 -0.03" />
     <xacro:property name="vertical_camera_orientation" value="0 ${radians(90)} 0" />
     <xacro:arg name="use_acoustic_modem" default="false" />
