Commit message: move vertical camera position to the back of bluerov

File: models/bluerov/urdf/bluerov_params.xacro (robot description, xacro)
@@ -21,5 +21,5 @@
     <xacro:property name="range_sensor_orientation" value="${radians(0)} ${radians(0)} ${radians(0)}" />
     <xacro:arg name="use_vertical_camera" default="false" />
-    <xacro:property name="vertical_camera_position" value="0.15 0 -0.08" />
+    <xacro:property name="vertical_camera_position" value="-0.145 0 -0.08" />
     <xacro:property name="vertical_camera_orientation" value="0 ${radians(90)} 0" />
     <xacro:arg name="use_front_camera" default="false" />
