Commit message: fixed wrong apriltag frame and set camera resolution

File: models/camera/urdf/camera_macro.xacro (robot description, xacro)
@@ -34,4 +34,9 @@
             <sensor name="$(arg vehicle_name)_${prefix}" type="camera">
                 <camera>
+                    <noise>
+                        <type>gaussian</type>
+                        <mean>0</mean>
+                        <stddev>0.1</stddev>
+                    </noise>
                     <camera_info_topic>$(arg vehicle_name)/${prefix}/camera_info</camera_info_topic>
                     <horizontal_fov>${horizontal_fov}</horizontal_fov>

File: models/camera/urdf/camera_params.xacro (robot description, xacro)
@@ -1,6 +1,6 @@
 <?xml version="1.0"?>
 <robot xmlns:xacro="http://www.ros.org/wiki/xacro">
-    <xacro:property name="width" value="640" />
-    <xacro:property name="height" value="480" />
+    <xacro:property name="width" value="1280" />
+    <xacro:property name="height" value="800" />
     <xacro:property name="fps" value="10" />
     <xacro:property name="horizontal_fov" value="1.2" />
